Commit message: modified file structure and plugins for easier addition of arms

File: urdf/robots/polysat_description/urdf/polysat_thrusters.xacro (robot description, xacro)
@@ -1,3 +1,44 @@
 <?xml version="1.0"?>
-<xacro:macro name="add_thruster">
-</xacro:macro>
+<robot xmlns:xacro="http://www.ros.org/wiki/xacro">
+  <xacro:macro name="thruster_macro" params="namespace thruster_id *origin">
+   <joint name="${namespace}/thruster_${thruster_id}_joint" type="fixed">
+     <xacro:insert_block name="origin"/>
+     <parent link="${namespace}/base_link"/>
+     <child link="${namespace}/thruster_${thruster_id}"/>
+   </joint>
+   <link name="${namespace}/thruster_${thruster_id}">
+     <xacro:box_inertial x="0" y="0" z="0" mass="0.0001">
+       <origin xyz="0 0 0" rpy="0 0 0"/>
+     </xacro:box_inertial>
+     <visual>
+       <origin rpy="0 0 0" xyz="0 0 0"/>
+     </visual>
+     <collision>
+       <geometry>
+         <cylinder length="0.0000001" radius="0.0000001"/>
+       </geometry>
+       <origin xyz="0 0 0" rpy="0 0 0"/>
+     </collision>
+   </link>
+   <gazebo>
+     <plugin name="${namespace}_${thruster_id}_thruster_model" filename="libsc_gazebo_thrust_plugin.so">
+       <thruster>
+         <linkName>${namespace}/thruster_${thruster_id}</linkName>
+         <jointName>${namespace}/thruster_${thruster_id}_joint</jointName>
+         <cmdTopic>${namespace}/thrusters/thruster_${thruster_id}</cmdTopic>
+         <angleTopic>${namespace}/thrusters/thruster_${thruster_id}_angle</angleTopic>
+         <enableAngle>false</enableAngle>
+       </thruster>
+     </plugin>
+   </gazebo>
+  </xacro:macro>
+  <xacro:macro name="box_inertial" params="x y z mass *origin">
+    <inertial>
+      <mass value="${mass}"/>
+      <xacro:insert_block name="origin"/>
+      <inertia ixx="${0.0833333 * mass * (y*y + z*z)}" ixy="0.0" ixz="0.0"
+               iyy="${0.0833333 * mass * (x*x + z*z)}" iyz="0.0"
+               izz="${0.0833333 * mass * (x*x + y*y)}"/>
+      </inertial>
+  </xacro:macro>
+</robot>

Commit message: Change world settings, removed grid. Check how to remove clouds faster

File: urdf/robots/polysat_description/urdf/polysat_thrusters.xacro (robot description, xacro)
@@ -37,4 +37,22 @@
       </plugin>
     </gazebo>
+    <!-- <gazebo>
+      <plugin name="${namespace}_${thruster_id}_thruster_model" filename="libLedPlugin.so">
+        <light>
+          <id>${namespace}/thruster_${thruster_id}/light</id>
+          <block>
+            <duration>1</duration>
+            <interval>1</interval>
+            <color>1 0.5 0.5</color>
+          </block>
+          <enable>true</enable>
+        </light>
+      </plugin>
+    </gazebo> -->
+    <!--gazebo reference="${namespace}/thruster_${thruster_id}">
+      <xacro:led_stripe name="light_${thruster_id}" range="30" linear="0.2" constant="0.1" quadratic="0.0025"
+        inner_angle="2.8" outer_angle="2.9"
+        pose="0 0 0 0 0 0"/>
+    </gazebo-->
     <gazebo reference="${namespace}/thruster_${thruster_id}">
       <selfCollide>false</selfCollide>
@@ -50,3 +68,23 @@
     </inertial>
   </xacro:macro>
+  <xacro:macro name="led_stripe" params="name pose range linear:=1 constant:=0 quadratic:=0 inner_angle outer_angle">
+    <light name="${name}" type="spot">
+      <pose>${pose}</pose>
+      <cast_shadows>1</cast_shadows>
+      <attenuation>
+        <range>${range}</range>
+        <linear>${linear}</linear>
+        <constant>${constant}</constant>
+        <quadratic>${quadratic}</quadratic>
+      </attenuation>
+      <diffuse>0.8 0.8 0.5 1</diffuse>
+      <specular>0.8 0.8 0.5 1</specular>
+      <spot>
+        <inner_angle>${inner_angle}</inner_angle>
+        <outer_angle>${outer_angle}</outer_angle>
+        <falloff>1</falloff>
+      </spot>
+      <direction>1 0 0</direction>
+    </light>
+  </xacro:macro>
 </robot>
