Commit message: Fixed thrusters and joints

File: urdf/robots/polysat_description/urdf/polysat_base.xacro (robot description, xacro)
@@ -1,6 +1,6 @@
 <?xml version="1.0"?>
-<robot xmlns:xacro="https://www.ros.org/wiki/xacro">
+<robot name="polysat" xmlns:xacro="https://www.ros.org/wiki/xacro">
   <!-- <xacro:property name="debug" default="false"/> -->
-  <xacro:property name="namespace" default="polysat"/>
+  <xacro:arg name="namespace" default="polysat"/>
   <xacro:include filename="$(find polysat_description)/urdf/polysat_thrusters.xacro"/>
   <xacro:macro name="polysat_base" params="namespace">
@@ -13,7 +13,7 @@
         <mass value="100.0"/>
         <inertia
-          ixx="1.0" ixy="0.0" ixz="0.0"
-          iyy="1.0" iyz="0.0"
-          izz="1.0"/>
+          ixx="10.0" ixy="0.0" ixz="0.0"
+          iyy="10.0" iyz="0.0"
+          izz="10.0"/>
       </inertial>
       <visual>
@@ -36,11 +36,52 @@
       <child link="$(arg namespace)/polysat_link"/>
     </joint>
-      <gazebo reference="$(arg namespace)/base_link">
+    <gazebo reference="$(arg namespace)/base_link">
       <gravity>0</gravity>
     </gazebo>
-    <!-- Add thrusters -->
+    <gazebo reference="$(arg namespace)/polysat_link">
+      <gravity>0</gravity>
+    </gazebo>
+    <gazebo>
+      <plugin name="gazebo_ros_control" filename="libgazebo_ros_control.so">
+        <robotNamespace>$(arg namespace)</robotNamespace>
+        <robotParam>$(arg namespace)</robotParam>
+      </plugin>
+    </gazebo>
+    <!-- Add maneuvering thrusters -->
     <xacro:thruster_macro namespace="${namespace}" thruster_id="0">
-      <origin xyz="0 0 0" rpy="0 0 0"/>
+      <origin xyz="0.5 0 0.5" rpy="0 0 0"/>
     </xacro:thruster_macro>
+    <xacro:thruster_macro namespace="${namespace}" thruster_id="1">
+      <origin xyz="-0.5 0 0.5" rpy="0 0 3.1415926535"/>
+    </xacro:thruster_macro>
+    <xacro:thruster_macro namespace="${namespace}" thruster_id="2">
+      <origin xyz="0.5 0 -0.5" rpy="0 0 0"/>
+    </xacro:thruster_macro>
+    <xacro:thruster_macro namespace="${namespace}" thruster_id="3">
+      <origin xyz="-0.5 0 -0.5" rpy="0 0 3.1415926535"/>
+    </xacro:thruster_macro>
+    <xacro:thruster_macro namespace="${namespace}" thruster_id="4">
+      <origin xyz="0 0.5 0.5" rpy="0 0 0"/>
+    </xacro:thruster_macro>
+    <xacro:thruster_macro namespace="${namespace}" thruster_id="5">
+      <origin xyz="0 -0.5 0.5" rpy="0 3.1415926535 0"/>
+    </xacro:thruster_macro>
+    <xacro:thruster_macro namespace="${namespace}" thruster_id="6">
+      <origin xyz="0 0.5 -0.5" rpy="0 0 0"/>
+    </xacro:thruster_macro>
+    <xacro:thruster_macro namespace="${namespace}" thruster_id="7">
+      <origin xyz="0 -0.5 -0.5" rpy="0 3.1415926535 0"/>
+    </xacro:thruster_macro>
+    <xacro:thruster_macro namespace="${namespace}" thruster_id="8">
+      <origin xyz="0.5 0 0.5" rpy="0 0 0"/>
+    </xacro:thruster_macro>
+    <xacro:thruster_macro namespace="${namespace}" thruster_id="9">
+      <origin xyz="0.5 0 -0.5" rpy="3.1415926535 0 0"/>
+    </xacro:thruster_macro>
+    <xacro:thruster_macro namespace="${namespace}" thruster_id="10">
+      <origin xyz="-0.5 0 0.5" rpy="0 0 0"/>
+    </xacro:thruster_macro>
+    <xacro:thruster_macro namespace="${namespace}" thruster_id="11">
+      <origin xyz="-0.5 0 -0.5" rpy="3.1415926535 0 0"/>
   </xacro:macro>
 </robot>

File: urdf/robots/polysat_description/urdf/polysat_thrusters.xacro (robot description, xacro)
@@ -2,34 +2,40 @@
 <robot xmlns:xacro="http://www.ros.org/wiki/xacro">
   <xacro:macro name="thruster_macro" params="namespace thruster_id *origin">
-   <joint name="${namespace}/thruster_${thruster_id}_joint" type="fixed">
-     <xacro:insert_block name="origin"/>
-     <parent link="${namespace}/base_link"/>
-     <child link="${namespace}/thruster_${thruster_id}"/>
-   </joint>
-   <link name="${namespace}/thruster_${thruster_id}">
-     <xacro:box_inertial x="0" y="0" z="0" mass="0.0001">
-       <origin xyz="0 0 0" rpy="0 0 0"/>
-     </xacro:box_inertial>
-     <visual>
-       <origin rpy="0 0 0" xyz="0 0 0"/>
-     </visual>
-     <collision>
-       <geometry>
-         <cylinder length="0.0000001" radius="0.0000001"/>
-       </geometry>
-       <origin xyz="0 0 0" rpy="0 0 0"/>
-     </collision>
-   </link>
-   <gazebo>
-     <plugin name="${namespace}_${thruster_id}_thruster_model" filename="libsc_gazebo_thrust_plugin.so">
-       <thruster>
-         <linkName>${namespace}/thruster_${thruster_id}</linkName>
-         <jointName>${namespace}/thruster_${thruster_id}_joint</jointName>
-         <cmdTopic>${namespace}/thrusters/thruster_${thruster_id}</cmdTopic>
-         <angleTopic>${namespace}/thrusters/thruster_${thruster_id}_angle</angleTopic>
-         <enableAngle>false</enableAngle>
-       </thruster>
-     </plugin>
-   </gazebo>
+    <link name="${namespace}/thruster_${thruster_id}">
+      <xacro:box_inertial x="0.001" y="0.001" z="0.001" mass="0.0001">
+        <origin xyz="0 0 0" rpy="0 0 0"/>
+      </xacro:box_inertial>
+      <visual>
+        <geometry>
+          <cylinder length="0.000001" radius="0.0000001"/>
+        </geometry>
+        <origin rpy="0 0 0" xyz="0 0 0"/>
+      </visual>
+      <collision>
+        <geometry>
+          <cylinder length="0.0000001" radius="0.0000001"/>
+        </geometry>
+        <origin xyz="0 0 0" rpy="0 0 0"/>
+      </collision>
+    </link>
+    <joint name="${namespace}/thruster_${thruster_id}_joint" type="continuous">
+      <xacro:insert_block name="origin"/>
+      <parent link="${namespace}/base_link"/>
+      <child link="${namespace}/thruster_${thruster_id}"/>
+    </joint>
+    <gazebo>
+      <plugin name="${namespace}_${thruster_id}_thruster_model" filename="libsc_gazebo_thrust_plugin.so">
+        <thruster>
+          <linkName>${namespace}/thruster_${thruster_id}</linkName>
+          <jointName>${namespace}/thruster_${thruster_id}_joint</jointName>
+          <cmdTopic>${namespace}/thrusters/thruster_${thruster_id}</cmdTopic>
+          <angleTopic>${namespace}/thrusters/thruster_${thruster_id}_angle</angleTopic>
+          <enableAngle>false</enableAngle>
+        </thruster>
+      </plugin>
+    </gazebo>
+   <gazebo reference="${namespace}/thruster_${thruster_id}">
+    <gravity>0</gravity>
+  </gazebo>
   </xacro:macro>
   <xacro:macro name="box_inertial" params="x y z mass *origin">
@@ -40,5 +46,5 @@
                iyy="${0.0833333 * mass * (x*x + z*z)}" iyz="0.0"
                izz="${0.0833333 * mass * (x*x + y*y)}"/>
-      </inertial>
+    </inertial>
   </xacro:macro>
 </robot>

Commit message: Added imu sensor to model

File: urdf/robots/polysat_description/urdf/polysat_base.xacro (robot description, xacro)
@@ -84,4 +84,14 @@
     <xacro:thruster_macro namespace="${namespace}" thruster_id="11">
       <origin xyz="-0.5 0 -0.5" rpy="3.1415926535 0 0"/>
-  </xacro:macro>
+    </xacro:thruster_macro>
+    <xacro:arg name="inertial_reference_frame" default="world"/>
+    <xacro:include filename="$(find sc_gazebo_plugins)/urdf/imu.xacro"/>
+    <!-- IMU  -->
+    <xacro:default_imu_macro
+      namespace="$(arg namespace)"
+      parent_link="$(arg namespace)/base_link"
+      inertial_reference_frame="$(arg inertial_reference_frame)">
+      <origin xyz="0 0 0" rpy="0 0 0"/>
+    </xacro:default_imu_macro>
+   </xacro:macro>
 </robot>

File: urdf/robots/polysat_description/urdf/polysat_robot.urdf.xacro (robot description, xacro)
@@ -3,5 +3,7 @@
   <xacro:arg name="namespace" default="polysat"/>
   <xacro:arg name="debug" default="false"/>
+  <xacro:arg name="inertial_reference_frame" default="world"/>
   <xacro:include filename="$(find polysat_description)/urdf/polysat_base.xacro"/>
   <xacro:polysat_base namespace="$(arg namespace)"/>
+  <!--xacro:include filename="$(find polysat_description)/urdf/polysat_sensors.xacro"/-->
 </robot>

File: urdf/robots/polysat_description/urdf/polysat_sensors.xacro (robot description, xacro)
@@ -1,4 +1,5 @@
 <?xml version="1.0"?>
 <robot xmlns:xacro="http://www.ros.org/wiki/xacro">
+  <xacro:include filename="$(find sc_gazebo_plugins)/urdf/imu.xacro"/>
   <!-- IMU  -->
   <xacro:default_imu_macro
@@ -8,2 +9,3 @@
     <origin xyz="0 0 0" rpy="0 0 0"/>
   </xacro:default_imu_macro>
+</robot>

Commit message: Fixed thruster joint issue

File: urdf/robots/polysat_description/urdf/polysat_base.xacro (robot description, xacro)
@@ -47,8 +47,8 @@
     </xacro:thruster_macro>
     <xacro:thruster_macro namespace="${namespace}" thruster_id="1">
-      <origin xyz="-0.5 0 0.5" rpy="0 0 3.1415926535"/>
+      <origin xyz="0.5 0 -0.5" rpy="0 0 0"/>
     </xacro:thruster_macro>
     <xacro:thruster_macro namespace="${namespace}" thruster_id="2">
-      <origin xyz="0.5 0 -0.5" rpy="0 0 0"/>
+      <origin xyz="-0.5 0 0.5" rpy="0 0 3.1415926535"/>
     </xacro:thruster_macro>
     <xacro:thruster_macro namespace="${namespace}" thruster_id="3">
@@ -56,26 +56,26 @@
     </xacro:thruster_macro>
     <xacro:thruster_macro namespace="${namespace}" thruster_id="4">
-      <origin xyz="0 0.5 0.5" rpy="0 0 0"/>
+      <origin xyz="0 0.5 0.5" rpy="0 -1.5707963268 0"/>
     </xacro:thruster_macro>
     <xacro:thruster_macro namespace="${namespace}" thruster_id="5">
-      <origin xyz="0 -0.5 0.5" rpy="0 3.1415926535 0"/>
+      <origin xyz="0 -0.5 0.5" rpy="0 -1.5707963268 0"/>
     </xacro:thruster_macro>
     <xacro:thruster_macro namespace="${namespace}" thruster_id="6">
-      <origin xyz="0 0.5 -0.5" rpy="0 0 0"/>
+      <origin xyz="0 0.5 -0.5" rpy="0 1.5707963268 0"/>
     </xacro:thruster_macro>
     <xacro:thruster_macro namespace="${namespace}" thruster_id="7">
-      <origin xyz="0 -0.5 -0.5" rpy="0 3.1415926535 0"/>
+      <origin xyz="0 -0.5 -0.5" rpy="0 1.5707963268 0"/>
     </xacro:thruster_macro>
     <xacro:thruster_macro namespace="${namespace}" thruster_id="8">
-      <origin xyz="0.5 0 0.5" rpy="0 0 0"/>
+      <origin xyz="0.5 0.5 0" rpy="0 0 0"/>
     </xacro:thruster_macro>
     <xacro:thruster_macro namespace="${namespace}" thruster_id="9">
-      <origin xyz="0.5 0 -0.5" rpy="3.1415926535 0 0"/>
+      <origin xyz="0.5 -0.5 0" rpy="0 0 0"/>
     </xacro:thruster_macro>
     <xacro:thruster_macro namespace="${namespace}" thruster_id="10">
-      <origin xyz="-0.5 0 0.5" rpy="0 0 0"/>
+      <origin xyz="-0.5 0.5 0" rpy="0 0 0"/>
     </xacro:thruster_macro>
     <xacro:thruster_macro namespace="${namespace}" thruster_id="11">
-      <origin xyz="-0.5 0 -0.5" rpy="3.1415926535 0 0"/>
+      <origin xyz="-0.5 -0.5 0" rpy="0 0 0"/>
     </xacro:thruster_macro>
     <xacro:arg name="inertial_reference_frame" default="world"/>

File: urdf/robots/polysat_description/urdf/polysat_thrusters.xacro (robot description, xacro)
@@ -23,4 +23,6 @@
       <parent link="${namespace}/base_link"/>
       <child link="${namespace}/thruster_${thruster_id}"/>
+      <axis xyz="1 0 0"/>
+      <limit effort="0" lower="0" upper="0" velocity="0"/>
     </joint>
     <gazebo>
@@ -35,4 +37,7 @@
       </plugin>
     </gazebo>
+    <gazebo reference="${namespace}/thruster_${thruster_id}">
+      <selfCollide>false</selfCollide>
+    </gazebo>
   </xacro:macro>
   <xacro:macro name="box_inertial" params="x y z mass *origin">

Commit message: Manual configuration nearly complete. Added all but strafe maneuvers

File: urdf/robots/polysat_description/urdf/polysat_base.xacro (robot description, xacro)
@@ -74,8 +74,8 @@
     </xacro:thruster_macro>
     <xacro:thruster_macro namespace="${namespace}" thruster_id="10">
-      <origin xyz="-0.5 0.5 0" rpy="0 0 0"/>
+      <origin xyz="-0.5 0.5 0" rpy="0 0 3.1415926535"/>
     </xacro:thruster_macro>
     <xacro:thruster_macro namespace="${namespace}" thruster_id="11">
-      <origin xyz="-0.5 -0.5 0" rpy="0 0 0"/>
+      <origin xyz="-0.5 -0.5 0" rpy="0 0 3.1415926535"/>
     </xacro:thruster_macro>
     <xacro:arg name="inertial_reference_frame" default="world"/>

Commit message: Added strafe thrusters and manual control mixing

File: urdf/robots/polysat_description/urdf/polysat_base.xacro (robot description, xacro)
@@ -79,4 +79,10 @@
       <origin xyz="-0.5 -0.5 0" rpy="0 0 3.1415926535"/>
     </xacro:thruster_macro>
+    <xacro:thruster_macro namespace="${namespace}" thruster_id="12">
+      <origin xyz="0 0.5 0" rpy="0 0 1.5707963268"/>
+    </xacro:thruster_macro>
+    <xacro:thruster_macro namespace="${namespace}" thruster_id="13">
+      <origin xyz="0 -0.5 0" rpy="0 0 -1.5707963268"/>
+    </xacro:thruster_macro>
     <xacro:arg name="inertial_reference_frame" default="world"/>
     <xacro:include filename="$(find sc_gazebo_plugins)/urdf/imu.xacro"/>

Commit message: y axis movement tuned for

File: urdf/robots/polysat_description/urdf/polysat_base.xacro (robot description, xacro)
@@ -11,5 +11,5 @@
       <inertial>
         <origin xyz="0 0 0" rpy="0 0 0"/>
-        <mass value="100.0"/>
+        <mass value="50.0"/>
         <inertia
           ixx="10.0" ixy="0.0" ixz="0.0"

Commit message: meh

File: urdf/robots/polysat_description/urdf/polysat_base.xacro (robot description, xacro)
@@ -22,4 +22,12 @@
           <box size="1.0 1.0 1.0"/>
         </geometry>
+        <material name="sat_mat">
+          <color rgba="1 0 1 1"/>
+        </material>
+        <!--plugin name="blink" filename="libsc_led_visual_plugin.so">
+          <color_a>1 0 0 1</color_a>
+          <color_b>1 0 0 0</color_b>
+          <period>1</period>
+        </plugin-->
       </visual>
       <collision>
@@ -94,4 +102,11 @@
       <origin xyz="0 0 0" rpy="0 0 0"/>
     </xacro:default_imu_macro>
+    <gazebo reference="$(arg namespace)/polysat_link">
+      <plugin name="blink" filename="libsc_led_visual_plugin.so">
+        <color_a>1 0 0 1</color_a>
+        <color_b>1 0 0 0</color_b>
+        <period>1</period>
+      </plugin>
+    </gazebo>
    </xacro:macro>
 </robot>

File: urdf/robots/polysat_description/urdf/polysat_thrusters.xacro (robot description, xacro)
@@ -50,9 +50,9 @@
       </plugin>
     </gazebo> -->
-    <!--gazebo reference="${namespace}/thruster_${thruster_id}">
-      <xacro:led_stripe name="light_${thruster_id}" range="30" linear="0.2" constant="0.1" quadratic="0.0025"
+    <gazebo reference="${namespace}/thruster_${thruster_id}">
+      <xacro:led_stripe name="light_${thruster_id}" range="1" linear="0.2" constant="0.1" quadratic="0.0025"
         inner_angle="2.8" outer_angle="2.9"
         pose="0 0 0 0 0 0"/>
-    </gazebo-->
+    </gazebo>
     <gazebo reference="${namespace}/thruster_${thruster_id}">
       <selfCollide>false</selfCollide>

Commit message: Added urdf sdf script and stl meshes

File: urdf/robots/polysat_description/urdf/polysat_base.xacro (robot description, xacro)
@@ -18,13 +18,13 @@
       </inertial>
       <visual>
-        <origin xyz="0 0 0" rpy="0 0 0"/>
+        <origin xyz="-0.5 1.0 -0.5" rpy="1.570796326794 0 0"/>
         <geometry>
-          <box size="1.0 1.0 1.0"/>
+          <mesh filename="file://$(find polysat_description)/meshes/Base.stl" scale="0.001 0.001 0.001"/>
         </geometry>
       </visual>
       <collision>
-        <origin xyz="0 0 0" rpy="0 0 0"/>
+        <origin xyz="-0.5 1.0 -0.5" rpy="1.570796326794 0 0"/>
         <geometry>
-          <box size="1.0 1.0 1.0"/>
+          <mesh filename="file://$(find polysat_description)/meshes/Base.stl" scale="0.001 0.001 0.001"/>
         </geometry>
       </collision>

File: urdf/robots/polysat_description/urdf/polysat_robot.urdf (robot description, URDF)
Before this commit: robot polysat, 18 links, 17 joints
Links:
- link polysat/polysat_link: geometry collision mesh filename=file:///home/carson/spaceship_ws/src/spacecraft_sim/urdf/ro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 scale=0.001 0.001 0.001; visual mesh filename=file:///home/carson/spaceship_ws/src/spacecraft_sim/urdf/ro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 scale=0.001 0.001 0.001

Commit message: Added first thruster nozzle. Need macro for easier config

File: urdf/robots/polysat_description/urdf/polysat_base.xacro (robot description, xacro)
@@ -30,4 +30,32 @@
       </collision>
     </link>
+    <!-- Add thruster meshes -->
+    <link name="$(arg namespace)/thruster__visual_link">
+      <inertial>
+        <origin xyz="0 0 0" rpy="0 0 0"/>
+        <mass value="0.00001"/>
+        <inertia
+          ixx="0.0001" ixy="0.0" ixz="0.0"
+          iyy="0.0001" iyz="0.0"
+          izz="0.0001"/>
+      </inertial>
+      <visual>
+        <origin xyz="0 0 0" rpy="0 0 0"/>
+        <geometry>
+          <mesh filename="file://$(find polysat_description)/meshes/thruster.stl" scale="0.001 0.001 0.001"/>
+        </geometry>
+      </visual>
+      <collision>
+        <origin xyz="0 0 0" rpy="0 0 0"/>
+        <geometry>
+          <mesh filename="file://$(find polysat_description)/meshes/thruster.stl" scale="0.001 0.001 0.001"/>
+        </geometry>
+      </collision>
+    </link>
+    <joint name="$(arg namespace)/thruster__visual_joint" type="fixed">
+      <origin xyz="0.5 0 0.5" rpy="0 0 0"/>
+      <parent link="$(arg namespace)/base_link"/>
+      <child link="$(arg namespace)/thruster__visual_link"/>
+    </joint>
     <!-- Connect dummy link to main link -->
     <joint name="$(arg namespace)/polysat_base_joint" type="fixed">

File: urdf/robots/polysat_description/urdf/polysat_robot.urdf (robot description, URDF)
Before this commit: robot polysat, 18 links, 17 joints
Links:
- added link polysat/thruster__visual_link, mass 0.00001; collision mesh filename=file:///home/carson/spaceship_ws/src/spacecraft_sim/urdf/ro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 scale=0.001 0.001 0.001; visual mesh filename=file:///home/carson/spaceship_ws/src/spacecraft_sim/urdf/ro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 scale=0.001 0.001 0.001
Joints:
- added joint polysat/thruster__visual_joint: type fixed, parent polysat/base_link, child polysat/thruster__visual_link, origin xyz=0.5 0 0.5 rpy=0 0 0

Commit message: Added positioning macros

File: urdf/robots/polysat_description/urdf/polysat_base.xacro (robot description, xacro)
@@ -4,4 +4,5 @@
   <xacro:arg name="namespace" default="polysat"/>
   <xacro:include filename="$(find polysat_description)/urdf/polysat_thrusters.xacro"/>
+  <xacro:include filename="$(find polysat_description)/urdf/polysat_thruster_visuals.xacro"/>
   <xacro:macro name="polysat_base" params="namespace">
     <!-- "Dummy base link to eliminate root link inertia warning -->
@@ -20,5 +21,5 @@
         <origin xyz="-0.5 1.0 -0.5" rpy="1.570796326794 0 0"/>
         <geometry>
-          <mesh filename="file://$(find polysat_description)/meshes/Base.stl" scale="0.001 0.001 0.001"/>
+          <mesh filename="file://$(find polysat_description)/meshes/base.stl" scale="0.001 0.001 0.001"/>
         </geometry>
       </visual>
@@ -26,9 +27,11 @@
         <origin xyz="-0.5 1.0 -0.5" rpy="1.570796326794 0 0"/>
         <geometry>
-          <mesh filename="file://$(find polysat_description)/meshes/Base.stl" scale="0.001 0.001 0.001"/>
+          <mesh filename="file://$(find polysat_description)/meshes/base.stl" scale="0.001 0.001 0.001"/>
         </geometry>
       </collision>
     </link>
-    <!-- Add thruster meshes -->
+    <xacro:thruster_visual_macro namespace="$(arg namespace)" thruster_id="0" x="${0.5-0.145}" y="${-0.15/2}" z="0.5" R="0" P="0" Y="0"/>
+    <xacro:thrust_plume_visual_macro namespace="$(arg namespace)" thruster_id="0" x="${0.5-0.235}" y="0.165" z="0.55" R="${pi/2}" P="0" Y="0"/>
+    <!-- Add thruster meshes >
     <link name="$(arg namespace)/thruster__visual_link">
       <inertial>
@@ -54,8 +57,8 @@
     </link>
     <joint name="$(arg namespace)/thruster__visual_joint" type="fixed">
-      <origin xyz="0.5 0 0.5" rpy="0 0 0"/>
+      <origin xyz="${0.5-0.15} ${-0.15/2} 0.5" rpy="0 0 0"/>
       <parent link="$(arg namespace)/base_link"/>
       <child link="$(arg namespace)/thruster__visual_link"/>
-    </joint>
+    </joint-->
     <!-- Connect dummy link to main link -->
     <joint name="$(arg namespace)/polysat_base_joint" type="fixed">

File: urdf/robots/polysat_description/urdf/polysat_robot.urdf (robot description, URDF)
Before this commit: robot polysat, 19 links, 18 joints
Links:
- removed link polysat/thruster__visual_link
- added link polysat/thrust_plume_0_visual, mass 0.0001; collision mesh filename=file:///home/carson/spaceship_ws/src/spacecraft_sim/urdf/ro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 scale=0.001 0.001 0.001; visual mesh filename=file:///home/carson/spaceship_ws/src/spacecraft_sim/urdf/ro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 scale=0.001 0.001 0.001
- added link polysat/thruster_0_visual, mass 0.0001; collision mesh filename=file:///home/carson/spaceship_ws/src/spacecraft_sim/urdf/ro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 scale=0.001 0.001 0.001; visual mesh filename=file:///home/carson/spaceship_ws/src/spacecraft_sim/urdf/ro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 scale=0.001 0.001 0.001
Joints:
- removed joint polysat/thruster__visual_joint
- added joint polysat/thrust_plume_0_visual_joint: type fixed, parent polysat/base_link, child polysat/thrust_plume_0_visual, origin xyz=0.265 0.165 0.55 rpy=1.5707963267948966 0 0
- added joint polysat/thruster_0_visual_joint: type fixed, parent polysat/base_link, child polysat/thruster_0_visual, origin xyz=0.355 -0.075 0.5 rpy=0 0 0
