Commit message: Modified thruster visual plugin to accept different thrusters, adding remaining visual thrusters, verified oberon7 arms will work with world-saved sdf

File: urdf/robots/polysat_description/urdf/polysat_base.xacro (robot description, xacro)
@@ -31,39 +31,4 @@
       </collision>
     </link>
-    <xacro:thruster_visual_macro namespace="$(arg namespace)" thruster_id="0" x="${0.5-0.145}" y="${-0.15/2}" z="0.5" R="0" P="0" Y="0"/>
-    <xacro:thrust_plume_visual_macro namespace="$(arg namespace)" thruster_id="0" x="${0.5-0.235}" y="0.165" z="0.55" R="${pi/2}" P="0" Y="0"/>
-    <!-- Add thruster meshes >
-    <link name="$(arg namespace)/thruster__visual_link">
-      <inertial>
-        <origin xyz="0 0 0" rpy="0 0 0"/>
-        <mass value="0.00001"/>
-        <inertia
-          ixx="0.0001" ixy="0.0" ixz="0.0"
-          iyy="0.0001" iyz="0.0"
-          izz="0.0001"/>
-      </inertial>
-      <visual>
-        <origin xyz="0 0 0" rpy="0 0 0"/>
-        <geometry>
-          <mesh filename="file://$(find polysat_description)/meshes/thruster.stl" scale="0.001 0.001 0.001"/>
-        </geometry>
-        <plugin name="blink" filename="libsc_led_visual_plugin.so">
-          <color_a>1 0 0 1</color_a>
-          <color_b>1 0 0 0</color_b>
-          <period>1</period>
-        </plugin>
-      </visual>
-      <collision>
-        <origin xyz="0 0 0" rpy="0 0 0"/>
-        <geometry>
-          <mesh filename="file://$(find polysat_description)/meshes/thruster.stl" scale="0.001 0.001 0.001"/>
-        </geometry>
-      </collision>
-    </link>
-    <joint name="$(arg namespace)/thruster__visual_joint" type="fixed">
-      <origin xyz="${0.5-0.15} ${-0.15/2} 0.5" rpy="0 0 0"/>
-      <parent link="$(arg namespace)/base_link"/>
-      <child link="$(arg namespace)/thruster__visual_link"/>
-    </joint-->
     <!-- Connect dummy link to main link -->
     <joint name="$(arg namespace)/polysat_base_joint" type="fixed">
@@ -72,10 +37,24 @@
       <child link="$(arg namespace)/polysat_link"/>
     </joint>
-    <gazebo>
-      <plugin name="gazebo_ros_control" filename="libgazebo_ros_control.so">
-        <robotNamespace>$(arg namespace)</robotNamespace>
-        <robotParam>$(arg namespace)</robotParam>
-      </plugin>
-    </gazebo>
+    <!-- Add thruster visuals -->
+    <!-- Top -->
+    <xacro:thruster_visual_macro namespace="$(arg namespace)" thruster_id="0" x="${-0.15/2}" y="${0.85}" z="0.5" R="0" P="0" Y="0"/>
+    <xacro:thrust_plume_visual_macro namespace="$(arg namespace)" thruster_id="0" x="${-0.17}" y="${1.095}" z="0.55" R="${pi/2}" P="0" Y="0"/>
+    <xacro:thruster_visual_macro namespace="$(arg namespace)" thruster_id="1" x="${-0.15/2}" y="${-1.0}" z="0.5" R="0" P="0" Y="0"/>
+    <xacro:thrust_plume_visual_macro namespace="$(arg namespace)" thruster_id="1" x="${-0.17}" y="${-0.755}" z="0.55" R="${pi/2}" P="0" Y="0"/>
+    <!-- Bottom -->
+    <xacro:thruster_visual_macro namespace="$(arg namespace)" thruster_id="2" x="${-0.15/2}" y="${1.0}" z="-0.5" R="${pi}" P="0" Y="0"/>
+    <xacro:thrust_plume_visual_macro namespace="$(arg namespace)" thruster_id="2" x="${-0.17}" y="${0.755}" z="-0.55" R="${-pi/2}" P="0" Y="0"/>
+    <xacro:thruster_visual_macro namespace="$(arg namespace)" thruster_id="3" x="${-0.15/2}" y="${-.85}" z="-0.5" R="${pi}" P="0" Y="0"/>
+    <xacro:thrust_plume_visual_macro namespace="$(arg namespace)" thruster_id="3" x="${-0.17}" y="${-1.095}" z="-0.55" R="${-pi/2}" P="0" Y="0"/>
+    <!-- Front -->
+    <xacro:thruster_visual_macro namespace="$(arg namespace)" thruster_id="4" x="${0.5}" y="${1.0}" z="0.0" R="0" P="${pi/2}" Y="0"/>
+    <xacro:thrust_plume_visual_macro namespace="$(arg namespace)" thruster_id="4" x="${0.5}" y="${0.755}" z="0.0" R="${0}" P="0" Y="${-pi/2}"/>
+    <xacro:thruster_visual_macro namespace="$(arg namespace)" thruster_id="5" x="${0.5}" y="${-.85}" z="0.0" R="${0}" P="${pi/2}" Y="0"/>
+    <xacro:thrust_plume_visual_macro namespace="$(arg namespace)" thruster_id="5" x="${0.5}" y="${-1.095}" z="0.0" R="${0}" P="0" Y="${-pi/2}"/>
+    <xacro:thruster_visual_macro namespace="$(arg namespace)" thruster_id="6" x="${0.5}" y="${0.0}" z="-0.5" R="${0}" P="${pi/2}" Y="0"/>
+    <xacro:thrust_plume_visual_macro namespace="$(arg namespace)" thruster_id="6" x="${0.5}" y="${0.0}" z="-0.55" R="${0}" P="0" Y="${-pi/2}"/>
+    <xacro:thruster_visual_macro namespace="$(arg namespace)" thruster_id="7" x="${0.5}" y="${0.0}" z="0.5" R="${0}" P="${pi/2}" Y="0"/>
+    <xacro:thrust_plume_visual_macro namespace="$(arg namespace)" thruster_id="7" x="${0.5}" y="${0.0}" z="0.55" R="${0}" P="0" Y="${-pi/2}"/>
     <!-- Add maneuvering thrusters -->
     <xacro:thruster_macro namespace="${namespace}" thruster_id="0">
@@ -121,4 +100,10 @@
       <origin xyz="0 -0.5 0" rpy="0 0 -1.5707963268"/>
     </xacro:thruster_macro>
+    <gazebo>
+      <plugin name="gazebo_ros_control" filename="libgazebo_ros_control.so">
+        <robotNamespace>$(arg namespace)</robotNamespace>
+        <robotParam>$(arg namespace)</robotParam>
+      </plugin>
+    </gazebo>
     <xacro:arg name="inertial_reference_frame" default="world"/>
     <xacro:include filename="$(find sc_gazebo_plugins)/urdf/imu.xacro"/>

File: urdf/robots/polysat_description/urdf/polysat_robot.urdf (robot description, URDF)
Before this commit: robot polysat, 20 links, 19 joints
Links:
- added link oberon7_l/base, mass 9.67467717018; collision mesh filename=package://oberon7_description/meshes/serial_arm/collision/B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; visual mesh filename=package://oberon7_description/meshes/serial_arm/visual/Base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
- added link oberon7_l/elbow_link, mass 10.3145088675; collision cylinder length=0.245312 radius=0.077562; visual mesh filename=package://oberon7_description/meshes/serial_arm/visual/Elbo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
- added link oberon7_l/end_effector, mass 3.46114581082; collision box size=0.074326 0.117427 0.114298; visual mesh filename=package://oberon7_description/meshes/parallel_gripper/visua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
- added link oberon7_l/finger_left, mass 0.879770511849; collision mesh filename=package://oberon7_description/meshes/parallel_gripper/visua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; visual mesh filename=package://oberon7_description/meshes/parallel_gripper/visua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
- added link oberon7_l/finger_right, mass 0.879770511849; collision mesh filename=package://oberon7_description/meshes/parallel_gripper/visua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; visual mesh filename=package://oberon7_description/meshes/parallel_gripper/visua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
- added link oberon7_l/finger_tip_left, mass 1.12550524054; collision mesh filename=package://oberon7_description/meshes/parallel_gripper/visua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; visual mesh filename=package://oberon7_description/meshes/parallel_gripper/visua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
- added link oberon7_l/finger_tip_right, mass 1.12550524054; collision mesh filename=package://oberon7_description/meshes/parallel_gripper/visua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; visual mesh filename=package://oberon7_description/meshes/parallel_gripper/visua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
- added link oberon7_l/forearm, mass 8.54626175585; collision cylinder length=0.334827 radius=0.0757275; visual mesh filename=package://oberon7_description/meshes/serial_arm/visual/Fore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
- added link oberon7_l/shoulder_link, mass 6.72225246901; collision cylinder length=0.239627 radius=0.068184; visual mesh filename=package://oberon7_description/meshes/serial_arm/visual/Shou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
- added link oberon7_l/upper_arm, mass 12.4443999072; collision cylinder length=0.616809 radius=0.0709445; visual mesh filename=package://oberon7_description/meshes/serial_arm/visual/Uppe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
- added link oberon7_l/wrist_link, mass 3.9024235777; collision cylinder length=0.219204 radius=0.065187; visual mesh filename=package://oberon7_description/meshes/serial_arm/visual/Wris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
- added link oberon7_r/base, mass 9.67467717018; collision mesh filename=package://oberon7_description/meshes/serial_arm/collision/B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; visual mesh filename=package://oberon7_description/meshes/serial_arm/visual/Base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
- added link oberon7_r/elbow_link, mass 10.3145088675; collision cylinder length=0.245312 radius=0.077562; visual mesh filename=package://oberon7_description/meshes/serial_arm/visual/Elbo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
- added link oberon7_r/end_effector, mass 3.46114581082; collision box size=0.074326 0.117427 0.114298; visual mesh filename=package://oberon7_description/meshes/parallel_gripper/visua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
- added link oberon7_r/finger_left, mass 0.879770511849; collision mesh filename=package://oberon7_description/meshes/parallel_gripper/visua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; visual mesh filename=package://oberon7_description/meshes/parallel_gripper/visua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
- added link oberon7_r/finger_right, mass 0.879770511849; collision mesh filename=package://oberon7_description/meshes/parallel_gripper/visua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; visual mesh filename=package://oberon7_description/meshes/parallel_gripper/visua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
- added link oberon7_r/finger_tip_left, mass 1.12550524054; collision mesh filename=package://oberon7_description/meshes/parallel_gripper/visua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; visual mesh filename=package://oberon7_description/meshes/parallel_gripper/visua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
- added link oberon7_r/finger_tip_right, mass 1.12550524054; collision mesh filename=package://oberon7_description/meshes/parallel_gripper/visua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; visual mesh filename=package://oberon7_description/meshes/parallel_gripper/visua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
- added link oberon7_r/forearm, mass 8.54626175585; collision cylinder length=0.334827 radius=0.0757275; visual mesh filename=package://oberon7_description/meshes/serial_arm/visual/Fore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
- added link oberon7_r/shoulder_link, mass 6.72225246901; collision cylinder length=0.239627 radius=0.068184; visual mesh filename=package://oberon7_description/meshes/serial_arm/visual/Shou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
- added link oberon7_r/upper_arm, mass 12.4443999072; collision cylinder length=0.616809 radius=0.0709445; visual mesh filename=package://oberon7_description/meshes/serial_arm/visual/Uppe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
- added link oberon7_r/wrist_link, mass 3.9024235777; collision cylinder length=0.219204 radius=0.065187; visual mesh filename=package://oberon7_description/meshes/serial_arm/visual/Wris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
Joints:
- added joint oberon7_l/azimuth: type revolute, parent oberon7_l/base, child oberon7_l/shoulder_link, axis 0 0 1, limit lower=-1.04719758 upper=1.04719758 effort=200 velocity=0.17
- added joint oberon7_l/elbow: type revolute, parent oberon7_l/upper_arm, child oberon7_l/elbow_link, origin xyz=0.55616 -0.01229 0 rpy=0 0 0, axis 0 0 1, limit lower=-1.4839 upper=1.04719758 effort=300 velocity=.13
- added joint oberon7_l/finger_left_joint: type revolute, parent oberon7_l/end_effector, child oberon7_l/finger_left, origin xyz=0.0444267 0.0391376 0 rpy=0 0 0, axis 0 0 1, limit lower=0 upper=1.04709283144 effort=3000 velocity=0.15
- added joint oberon7_l/finger_right_joint: type revolute, parent oberon7_l/end_effector, child oberon7_l/finger_right, origin xyz=0.0444267 -0.0391376 0 rpy=3.14159265359 3.14159265359 3.14159265359, axis 0 0 -1, limit lower=0 upper=1.04709283144 effort=3000 velocity=0.15
- added joint oberon7_l/finger_tip_left_joint: type revolute, parent oberon7_l/finger_left, child oberon7_l/finger_tip_left, origin xyz=0.06431 0 0 rpy=3.14159265359 0 0, axis 0 0 1, limit lower=0 upper=0 effort=0 velocity=0
- added joint oberon7_l/finger_tip_right_joint: type revolute, parent oberon7_l/finger_right, child oberon7_l/finger_tip_right, origin xyz=0.06431 0 0 rpy=0 0 0, axis 0 0 1, limit lower=0 upper=0 effort=0 velocity=0
- added joint oberon7_l/pitch: type revolute, parent oberon7_l/forearm, child oberon7_l/wrist_link, origin xyz=0 0 0.31595760629823427 rpy=-1.57079632679 -1.57079632679 0, axis 0 0 1, limit lower=-1.57079637 upper=1.57079637 effort=200 velocity=.26
- added joint oberon7_l/roll: type revolute, parent oberon7_l/elbow_link, child oberon7_l/forearm, origin xyz=0.1349014 -0.1936267 0 rpy=1.57079632679 0 0, axis 0 0 1, limit lower=-2.356194555 upper=2.356194555 effort=200 velocity=.085
- added joint oberon7_l/shoulder: type revolute, parent oberon7_l/shoulder_link, child oberon7_l/upper_arm, origin xyz=0.06955 0.00015 0.01536 rpy=1.57079632679 0 0, axis 0 0 1, limit lower=-0.8591 upper=0.6856 effort=5000 velocity=0.17
- added joint oberon7_l/wrist: type continuous, parent oberon7_l/wrist_link, child oberon7_l/end_effector, origin xyz=0.19304 0 0 rpy=0 0 0, axis 1 0 0
- added joint oberon7_l_anchor: type fixed, parent polysat/base_link, child oberon7_l/base, origin xyz=0 -1.5 0 rpy=1.5707963268 0 0
- added joint oberon7_r/azimuth: type revolute, parent oberon7_r/base, child oberon7_r/shoulder_link, axis 0 0 1, limit lower=-1.04719758 upper=1.04719758 effort=200 velocity=0.17
- added joint oberon7_r/elbow: type revolute, parent oberon7_r/upper_arm, child oberon7_r/elbow_link, origin xyz=0.55616 -0.01229 0 rpy=0 0 0, axis 0 0 1, limit lower=-1.4839 upper=1.04719758 effort=300 velocity=.13
- added joint oberon7_r/finger_left_joint: type revolute, parent oberon7_r/end_effector, child oberon7_r/finger_left, origin xyz=0.0444267 0.0391376 0 rpy=0 0 0, axis 0 0 1, limit lower=0 upper=1.04709283144 effort=3000 velocity=0.15
- added joint oberon7_r/finger_right_joint: type revolute, parent oberon7_r/end_effector, child oberon7_r/finger_right, origin xyz=0.0444267 -0.0391376 0 rpy=3.14159265359 3.14159265359 3.14159265359, axis 0 0 -1, limit lower=0 upper=1.04709283144 effort=3000 velocity=0.15
- added joint oberon7_r/finger_tip_left_joint: type revolute, parent oberon7_r/finger_left, child oberon7_r/finger_tip_left, origin xyz=0.06431 0 0 rpy=3.14159265359 0 0, axis 0 0 1, limit lower=0 upper=0 effort=0 velocity=0
- added joint oberon7_r/finger_tip_right_joint: type revolute, parent oberon7_r/finger_right, child oberon7_r/finger_tip_right, origin xyz=0.06431 0 0 rpy=0 0 0, axis 0 0 1, limit lower=0 upper=0 effort=0 velocity=0
- added joint oberon7_r/pitch: type revolute, parent oberon7_r/forearm, child oberon7_r/wrist_link, origin xyz=0 0 0.31595760629823427 rpy=-1.57079632679 -1.57079632679 0, axis 0 0 1, limit lower=-1.57079637 upper=1.57079637 effort=200 velocity=.26
- added joint oberon7_r/roll: type revolute, parent oberon7_r/elbow_link, child oberon7_r/forearm, origin xyz=0.1349014 -0.1936267 0 rpy=1.57079632679 0 0, axis 0 0 1, limit lower=-2.356194555 upper=2.356194555 effort=200 velocity=.085
- added joint oberon7_r/shoulder: type revolute, parent oberon7_r/shoulder_link, child oberon7_r/upper_arm, origin xyz=0.06955 0.00015 0.01536 rpy=1.57079632679 0 0, axis 0 0 1, limit lower=-0.8591 upper=0.6856 effort=5000 velocity=0.17
- added joint oberon7_r/wrist: type continuous, parent oberon7_r/wrist_link, child oberon7_r/end_effector, origin xyz=0.19304 0 0 rpy=0 0 0, axis 1 0 0
- added joint oberon7_r_anchor: type fixed, parent polysat/base_link, child oberon7_r/base, origin xyz=0 1.5 0 rpy=-1.5707963268 0 0

File: urdf/robots/polysat_description/urdf/polysat_robot.urdf.xacro (robot description, xacro)
@@ -17,5 +17,4 @@
     <xacro:arg name="transmission_hw_interface" default="hardware_interface/EffortJointInterface"/>
   </xacro:if>
-  <!--
   <xacro:oberon7_arm transmission_hw_interface="$(arg transmission_hw_interface)" namespace="oberon7_r"/>
   <xacro:oberon7_arm transmission_hw_interface="$(arg transmission_hw_interface)" namespace="oberon7_l"/>
@@ -30,4 +29,3 @@
     <origin rpy="1.5707963268 0 0" xyz="0 -1.5 0"/>
   </joint>
-  -->
 </robot>

File: urdf/robots/polysat_description/urdf/polysat_thruster_visuals.xacro (robot description, xacro)
@@ -35,9 +35,13 @@
           <mesh filename="file://$(find polysat_description)/meshes/thrust_plume.stl" scale="0.001 0.001 0.001"/>
         </geometry>
+        <plugin filename="libsc_thrust_visual_plugin.so" name="thrust_visual_${thruster_id}">
+          <thrust_color>1 0 0 1</thrust_color>
+          <thruster_number>${thruster_id}</thruster_number>
+        </plugin>
       </visual>
       <collision>
         <origin xyz="0 0 0" rpy="0 0 0"/>
         <geometry>
-          <mesh filename="file://$(find polysat_description)/meshes/thrust_plume.stl" scale="0.001 0.001 0.001"/>
+          <box size="0.0001 0.0001 0.0001"/>
         </geometry>
       </collision>
