Commit message: Finish python script for sdfs

File: urdf/robots/polysat_description/urdf/polysat_base.xacro (robot description, xacro)
@@ -39,31 +39,31 @@
     <!-- Add thruster visuals -->
     <!-- Top -->
-    <xacro:thruster_visual_macro namespace="$(arg namespace)" thruster_id="0" x="${-0.15/2}" y="${0.85}" z="0.5" R="0" P="0" Y="0"/>
-    <xacro:thrust_plume_visual_macro namespace="$(arg namespace)" thruster_id="0" x="${-0.17}" y="${1.095}" z="0.55" R="${pi/2}" P="0" Y="0"/>
-    <xacro:thruster_visual_macro namespace="$(arg namespace)" thruster_id="1" x="${-0.15/2}" y="${-1.0}" z="0.5" R="0" P="0" Y="0"/>
-    <xacro:thrust_plume_visual_macro namespace="$(arg namespace)" thruster_id="1" x="${-0.17}" y="${-0.755}" z="0.55" R="${pi/2}" P="0" Y="0"/>
+    <xacro:thruster_visual_macro namespace="$(arg namespace)" thruster_id="5" x="${-0.15/2}" y="${0.85}" z="0.5" R="0" P="0" Y="0"/>
+    <xacro:thrust_plume_visual_macro namespace="$(arg namespace)" thruster_id="5" x="${-0.17}" y="${1.095}" z="0.55" R="${pi/2}" P="0" Y="0"/>
+    <xacro:thruster_visual_macro namespace="$(arg namespace)" thruster_id="4" x="${-0.15/2}" y="${-1.0}" z="0.5" R="0" P="0" Y="0"/>
+    <xacro:thrust_plume_visual_macro namespace="$(arg namespace)" thruster_id="4" x="${-0.17}" y="${-0.755}" z="0.55" R="${pi/2}" P="0" Y="0"/>
     <!-- Bottom -->
-    <xacro:thruster_visual_macro namespace="$(arg namespace)" thruster_id="2" x="${-0.15/2}" y="${1.0}" z="-0.5" R="${pi}" P="0" Y="0"/>
-    <xacro:thrust_plume_visual_macro namespace="$(arg namespace)" thruster_id="2" x="${-0.17}" y="${0.755}" z="-0.55" R="${-pi/2}" P="0" Y="0"/>
-    <xacro:thruster_visual_macro namespace="$(arg namespace)" thruster_id="3" x="${-0.15/2}" y="${-.85}" z="-0.5" R="${pi}" P="0" Y="0"/>
-    <xacro:thrust_plume_visual_macro namespace="$(arg namespace)" thruster_id="3" x="${-0.17}" y="${-1.095}" z="-0.55" R="${-pi/2}" P="0" Y="0"/>
+    <xacro:thruster_visual_macro namespace="$(arg namespace)" thruster_id="6" x="${-0.15/2}" y="${1.0}" z="-0.5" R="${pi}" P="0" Y="0"/>
+    <xacro:thrust_plume_visual_macro namespace="$(arg namespace)" thruster_id="6" x="${-0.17}" y="${0.755}" z="-0.55" R="${-pi/2}" P="0" Y="0"/>
+    <xacro:thruster_visual_macro namespace="$(arg namespace)" thruster_id="7" x="${-0.15/2}" y="${-.85}" z="-0.5" R="${pi}" P="0" Y="0"/>
+    <xacro:thrust_plume_visual_macro namespace="$(arg namespace)" thruster_id="7" x="${-0.17}" y="${-1.095}" z="-0.55" R="${-pi/2}" P="0" Y="0"/>
     <!-- Front -->
-    <xacro:thruster_visual_macro namespace="$(arg namespace)" thruster_id="4" x="${0.5}" y="${0.85}" z="${0.15/2}" R="0" P="${pi/2}" Y="0"/>
-    <xacro:thrust_plume_visual_macro namespace="$(arg namespace)" thruster_id="4" x="${0.55}" y="${1.095}" z="-0.16" R="${0}" P="0" Y="${-pi/2}"/>
-    <xacro:thruster_visual_macro namespace="$(arg namespace)" thruster_id="5" x="${0.5}" y="${-1.0}" z="${0.15/2}" R="${0}" P="${pi/2}" Y="0"/>
-    <xacro:thrust_plume_visual_macro namespace="$(arg namespace)" thruster_id="5" x="${0.55}" y="${-0.76}" z="-0.17" R="${0}" P="0" Y="${-pi/2}"/>
-    <xacro:thruster_visual_macro namespace="$(arg namespace)" thruster_id="6" x="${0.5}" y="${-0.15/2}" z="-0.35" R="${0}" P="${pi/2}" Y="0"/>
-    <xacro:thrust_plume_visual_macro namespace="$(arg namespace)" thruster_id="6" x="${0.55}" y="${0.17}" z="-0.59" R="${0}" P="0" Y="${-pi/2}"/>
-    <xacro:thruster_visual_macro namespace="$(arg namespace)" thruster_id="7" x="${0.5}" y="${-0.15/2}" z="0.5" R="${0}" P="${pi/2}" Y="0"/>
-    <xacro:thrust_plume_visual_macro namespace="$(arg namespace)" thruster_id="7" x="${0.55}" y="${0.17}" z="0.26" R="${0}" P="0" Y="${-pi/2}"/>
+    <xacro:thruster_visual_macro namespace="$(arg namespace)" thruster_id="8" x="${0.5}" y="${0.85}" z="${0.15/2}" R="0" P="${pi/2}" Y="0"/>
+    <xacro:thrust_plume_visual_macro namespace="$(arg namespace)" thruster_id="8" x="${0.55}" y="${1.095}" z="-0.16" R="${0}" P="0" Y="${-pi/2}"/>
+    <xacro:thruster_visual_macro namespace="$(arg namespace)" thruster_id="9" x="${0.5}" y="${-1.0}" z="${0.15/2}" R="${0}" P="${pi/2}" Y="0"/>
+    <xacro:thrust_plume_visual_macro namespace="$(arg namespace)" thruster_id="9" x="${0.55}" y="${-0.76}" z="-0.17" R="${0}" P="0" Y="${-pi/2}"/>
+    <xacro:thruster_visual_macro namespace="$(arg namespace)" thruster_id="1" x="${0.5}" y="${-0.15/2}" z="-0.35" R="${0}" P="${pi/2}" Y="0"/>
+    <xacro:thrust_plume_visual_macro namespace="$(arg namespace)" thruster_id="1" x="${0.55}" y="${0.17}" z="-0.59" R="${0}" P="0" Y="${-pi/2}"/>
+    <xacro:thruster_visual_macro namespace="$(arg namespace)" thruster_id="0" x="${0.5}" y="${-0.15/2}" z="0.5" R="${0}" P="${pi/2}" Y="0"/>
+    <xacro:thrust_plume_visual_macro namespace="$(arg namespace)" thruster_id="0" x="${0.55}" y="${0.17}" z="0.26" R="${0}" P="0" Y="${-pi/2}"/>
     <!-- Back -->
-    <xacro:thruster_visual_macro namespace="$(arg namespace)" thruster_id="8" x="${-0.5}" y="${0.85}" z="${-0.15/2}" R="0" P="${-pi/2}" Y="0"/>
-    <xacro:thrust_plume_visual_macro namespace="$(arg namespace)" thruster_id="8" x="${-0.55}" y="${0.76}" z="-0.16" R="${0}" P="0" Y="${pi/2}"/>
-    <xacro:thruster_visual_macro namespace="$(arg namespace)" thruster_id="9" x="${-0.5}" y="${-1.0}" z="${-0.15/2}" R="${0}" P="${-pi/2}" Y="0"/>
-    <xacro:thrust_plume_visual_macro namespace="$(arg namespace)" thruster_id="9" x="${-0.55}" y="${-1.095}" z="-0.17" R="${0}" P="0" Y="${pi/2}"/>
-    <xacro:thruster_visual_macro namespace="$(arg namespace)" thruster_id="10" x="${-0.5}" y="${-0.15/2}" z="-0.5" R="${0}" P="${-pi/2}" Y="0"/>
-    <xacro:thrust_plume_visual_macro namespace="$(arg namespace)" thruster_id="10" x="${-0.55}" y="${-0.17}" z="-0.59" R="${0}" P="0" Y="${pi/2}"/>
-    <xacro:thruster_visual_macro namespace="$(arg namespace)" thruster_id="11" x="${-0.5}" y="${-0.15/2}" z="0.35" R="${0}" P="${-pi/2}" Y="0"/>
-    <xacro:thrust_plume_visual_macro namespace="$(arg namespace)" thruster_id="11" x="${-0.55}" y="${-0.17}" z="0.26" R="${0}" P="0" Y="${pi/2}"/>
+    <xacro:thruster_visual_macro namespace="$(arg namespace)" thruster_id="10" x="${-0.5}" y="${0.85}" z="${-0.15/2}" R="0" P="${-pi/2}" Y="0"/>
+    <xacro:thrust_plume_visual_macro namespace="$(arg namespace)" thruster_id="10" x="${-0.55}" y="${0.76}" z="-0.16" R="${0}" P="0" Y="${pi/2}"/>
+    <xacro:thruster_visual_macro namespace="$(arg namespace)" thruster_id="11" x="${-0.5}" y="${-1.0}" z="${-0.15/2}" R="${0}" P="${-pi/2}" Y="0"/>
+    <xacro:thrust_plume_visual_macro namespace="$(arg namespace)" thruster_id="11" x="${-0.55}" y="${-1.095}" z="-0.17" R="${0}" P="0" Y="${pi/2}"/>
+    <xacro:thruster_visual_macro namespace="$(arg namespace)" thruster_id="3" x="${-0.5}" y="${-0.15/2}" z="-0.5" R="${0}" P="${-pi/2}" Y="0"/>
+    <xacro:thrust_plume_visual_macro namespace="$(arg namespace)" thruster_id="3" x="${-0.55}" y="${-0.17}" z="-0.59" R="${0}" P="0" Y="${pi/2}"/>
+    <xacro:thruster_visual_macro namespace="$(arg namespace)" thruster_id="2" x="${-0.5}" y="${-0.15/2}" z="0.35" R="${0}" P="${-pi/2}" Y="0"/>
+    <xacro:thrust_plume_visual_macro namespace="$(arg namespace)" thruster_id="2" x="${-0.55}" y="${-0.17}" z="0.26" R="${0}" P="0" Y="${pi/2}"/>
     <!-- Sides -->
     <xacro:thruster_visual_macro namespace="$(arg namespace)" thruster_id="12" x="${-0.15/2}" y="${-1.0}" z="${-0.15/2}" R="${pi/2}" P="${0}" Y="0"/>

File: urdf/robots/polysat_description/urdf/polysat_robot.urdf.xacro (robot description, xacro)
@@ -22,10 +22,10 @@
     <parent link="$(arg namespace)/base_link"/>
     <child link="oberon7_r/base"/>
-    <origin rpy="-1.5707963268 0 0" xyz="0 1.5 0"/>
+    <origin rpy="-1.5707963268 0 0" xyz="0.5 1.06 -0.25"/>
   </joint>
   <joint name="oberon7_l_anchor" type="fixed">
     <parent link="$(arg namespace)/base_link"/>
     <child link="oberon7_l/base"/>
-    <origin rpy="1.5707963268 0 0" xyz="0 -1.5 0"/>
+    <origin rpy="1.5707963268 0 0" xyz="0.5 -1.06 -0.25"/>
   </joint>
 </robot>

Commit message: Not yet loading controllers...

File: urdf/robots/polysat_description/urdf/polysat_base.xacro (robot description, xacro)
@@ -39,15 +39,15 @@
     <!-- Add thruster visuals -->
     <!-- Top -->
-    <xacro:thruster_visual_macro namespace="$(arg namespace)" thruster_id="5" x="${-0.15/2}" y="${0.85}" z="0.5" R="0" P="0" Y="0"/>
+    <!--<xacro:thruster_visual_macro namespace="$(arg namespace)" thruster_id="5" x="${-0.15/2}" y="${0.85}" z="0.5" R="0" P="0" Y="0"/>
     <xacro:thrust_plume_visual_macro namespace="$(arg namespace)" thruster_id="5" x="${-0.17}" y="${1.095}" z="0.55" R="${pi/2}" P="0" Y="0"/>
     <xacro:thruster_visual_macro namespace="$(arg namespace)" thruster_id="4" x="${-0.15/2}" y="${-1.0}" z="0.5" R="0" P="0" Y="0"/>
-    <xacro:thrust_plume_visual_macro namespace="$(arg namespace)" thruster_id="4" x="${-0.17}" y="${-0.755}" z="0.55" R="${pi/2}" P="0" Y="0"/>
+    <xacro:thrust_plume_visual_macro namespace="$(arg namespace)" thruster_id="4" x="${-0.17}" y="${-0.755}" z="0.55" R="${pi/2}" P="0" Y="0"/-->
     <!-- Bottom -->
-    <xacro:thruster_visual_macro namespace="$(arg namespace)" thruster_id="6" x="${-0.15/2}" y="${1.0}" z="-0.5" R="${pi}" P="0" Y="0"/>
+    <!--<xacro:thruster_visual_macro namespace="$(arg namespace)" thruster_id="6" x="${-0.15/2}" y="${1.0}" z="-0.5" R="${pi}" P="0" Y="0"/>
     <xacro:thrust_plume_visual_macro namespace="$(arg namespace)" thruster_id="6" x="${-0.17}" y="${0.755}" z="-0.55" R="${-pi/2}" P="0" Y="0"/>
     <xacro:thruster_visual_macro namespace="$(arg namespace)" thruster_id="7" x="${-0.15/2}" y="${-.85}" z="-0.5" R="${pi}" P="0" Y="0"/>
-    <xacro:thrust_plume_visual_macro namespace="$(arg namespace)" thruster_id="7" x="${-0.17}" y="${-1.095}" z="-0.55" R="${-pi/2}" P="0" Y="0"/>
+    <xacro:thrust_plume_visual_macro namespace="$(arg namespace)" thruster_id="7" x="${-0.17}" y="${-1.095}" z="-0.55" R="${-pi/2}" P="0" Y="0"/-->
     <!-- Front -->
-    <xacro:thruster_visual_macro namespace="$(arg namespace)" thruster_id="8" x="${0.5}" y="${0.85}" z="${0.15/2}" R="0" P="${pi/2}" Y="0"/>
+    <!--<xacro:thruster_visual_macro namespace="$(arg namespace)" thruster_id="8" x="${0.5}" y="${0.85}" z="${0.15/2}" R="0" P="${pi/2}" Y="0"/>
     <xacro:thrust_plume_visual_macro namespace="$(arg namespace)" thruster_id="8" x="${0.55}" y="${1.095}" z="-0.16" R="${0}" P="0" Y="${-pi/2}"/>
     <xacro:thruster_visual_macro namespace="$(arg namespace)" thruster_id="9" x="${0.5}" y="${-1.0}" z="${0.15/2}" R="${0}" P="${pi/2}" Y="0"/>
@@ -56,7 +56,7 @@
     <xacro:thrust_plume_visual_macro namespace="$(arg namespace)" thruster_id="1" x="${0.55}" y="${0.17}" z="-0.59" R="${0}" P="0" Y="${-pi/2}"/>
     <xacro:thruster_visual_macro namespace="$(arg namespace)" thruster_id="0" x="${0.5}" y="${-0.15/2}" z="0.5" R="${0}" P="${pi/2}" Y="0"/>
-    <xacro:thrust_plume_visual_macro namespace="$(arg namespace)" thruster_id="0" x="${0.55}" y="${0.17}" z="0.26" R="${0}" P="0" Y="${-pi/2}"/>
+    <xacro:thrust_plume_visual_macro namespace="$(arg namespace)" thruster_id="0" x="${0.55}" y="${0.17}" z="0.26" R="${0}" P="0" Y="${-pi/2}"/-->
     <!-- Back -->
-    <xacro:thruster_visual_macro namespace="$(arg namespace)" thruster_id="10" x="${-0.5}" y="${0.85}" z="${-0.15/2}" R="0" P="${-pi/2}" Y="0"/>
+    <!--<xacro:thruster_visual_macro namespace="$(arg namespace)" thruster_id="10" x="${-0.5}" y="${0.85}" z="${-0.15/2}" R="0" P="${-pi/2}" Y="0"/>
     <xacro:thrust_plume_visual_macro namespace="$(arg namespace)" thruster_id="10" x="${-0.55}" y="${0.76}" z="-0.16" R="${0}" P="0" Y="${pi/2}"/>
     <xacro:thruster_visual_macro namespace="$(arg namespace)" thruster_id="11" x="${-0.5}" y="${-1.0}" z="${-0.15/2}" R="${0}" P="${-pi/2}" Y="0"/>
@@ -65,10 +65,10 @@
     <xacro:thrust_plume_visual_macro namespace="$(arg namespace)" thruster_id="3" x="${-0.55}" y="${-0.17}" z="-0.59" R="${0}" P="0" Y="${pi/2}"/>
     <xacro:thruster_visual_macro namespace="$(arg namespace)" thruster_id="2" x="${-0.5}" y="${-0.15/2}" z="0.35" R="${0}" P="${-pi/2}" Y="0"/>
-    <xacro:thrust_plume_visual_macro namespace="$(arg namespace)" thruster_id="2" x="${-0.55}" y="${-0.17}" z="0.26" R="${0}" P="0" Y="${pi/2}"/>
+    <xacro:thrust_plume_visual_macro namespace="$(arg namespace)" thruster_id="2" x="${-0.55}" y="${-0.17}" z="0.26" R="${0}" P="0" Y="${pi/2}"/-->
     <!-- Sides -->
-    <xacro:thruster_visual_macro namespace="$(arg namespace)" thruster_id="12" x="${-0.15/2}" y="${-1.0}" z="${-0.15/2}" R="${pi/2}" P="${0}" Y="0"/>
+    <!--<xacro:thruster_visual_macro namespace="$(arg namespace)" thruster_id="12" x="${-0.15/2}" y="${-1.0}" z="${-0.15/2}" R="${pi/2}" P="${0}" Y="0"/>
     <xacro:thrust_plume_visual_macro namespace="$(arg namespace)" thruster_id="12" x="${0.17}" y="${-1.05}" z="-0.17" R="${0}" P="0" Y="${pi}"/>
     <xacro:thruster_visual_macro namespace="$(arg namespace)" thruster_id="13" x="${-0.15/2}" y="${1.0}" z="${0.15/2}" R="${-pi/2}" P="${0}" Y="${0}"/>
-    <xacro:thrust_plume_visual_macro namespace="$(arg namespace)" thruster_id="13" x="${0.17}" y="${1.05}" z="0.17" R="${0}" P="${pi}" Y="${0}"/>
+    <xacro:thrust_plume_visual_macro namespace="$(arg namespace)" thruster_id="13" x="${0.17}" y="${1.05}" z="0.17" R="${0}" P="${pi}" Y="${0}"/-->
     <!-- Add maneuvering thrusters -->
     <xacro:thruster_macro namespace="${namespace}" thruster_id="0">

File: urdf/robots/polysat_description/urdf/polysat_thrusters.xacro (robot description, xacro)
@@ -3,7 +3,11 @@
   <xacro:macro name="thruster_macro" params="namespace thruster_id *origin">
     <link name="${namespace}/thruster_${thruster_id}">
-      <xacro:box_inertial x="0.001" y="0.001" z="0.001" mass="0.0001">
+      <inertial>
         <origin xyz="0 0 0" rpy="0 0 0"/>
-      </xacro:box_inertial>
+        <mass value="0.001"/>
+        <inertia ixx="0.001" ixy="0.0" ixz="0.0"
+                 iyy="0.001" iyz="0.0"
+                 izz="0.001"/>
+      </inertial>
       <visual>
         <geometry>
@@ -37,54 +41,7 @@
       </plugin>
     </gazebo>
-    <!-- <gazebo>
-      <plugin name="${namespace}_${thruster_id}_thruster_model" filename="libLedPlugin.so">
-        <light>
-          <id>${namespace}/thruster_${thruster_id}/light</id>
-          <block>
-            <duration>1</duration>
-            <interval>1</interval>
-            <color>1 0.5 0.5</color>
-          </block>
-          <enable>true</enable>
-        </light>
-      </plugin>
-    </gazebo> -->
-    <!--gazebo reference="${namespace}/thruster_${thruster_id}">
-      <xacro:led_stripe name="light_${thruster_id}" range="30" linear="0.2" constant="0.1" quadratic="0.0025"
-        inner_angle="2.8" outer_angle="2.9"
-        pose="0 0 0 0 0 0"/>
-    </gazebo-->
     <gazebo reference="${namespace}/thruster_${thruster_id}">
       <selfCollide>false</selfCollide>
     </gazebo>
   </xacro:macro>
-  <xacro:macro name="box_inertial" params="x y z mass *origin">
-    <inertial>
-      <mass value="${mass}"/>
-      <xacro:insert_block name="origin"/>
-      <inertia ixx="${0.0833333 * mass * (y*y + z*z)}" ixy="0.0" ixz="0.0"
-               iyy="${0.0833333 * mass * (x*x + z*z)}" iyz="0.0"
-               izz="${0.0833333 * mass * (x*x + y*y)}"/>
-    </inertial>
-  </xacro:macro>
-  <xacro:macro name="led_stripe" params="name pose range linear:=1 constant:=0 quadratic:=0 inner_angle outer_angle">
-    <light name="${name}" type="spot">
-      <pose>${pose}</pose>
-      <cast_shadows>1</cast_shadows>
-      <attenuation>
-        <range>${range}</range>
-        <linear>${linear}</linear>
-        <constant>${constant}</constant>
-        <quadratic>${quadratic}</quadratic>
-      </attenuation>
-      <diffuse>0.8 0.8 0.5 1</diffuse>
-      <specular>0.8 0.8 0.5 1</specular>
-      <spot>
-        <inner_angle>${inner_angle}</inner_angle>
-        <outer_angle>${outer_angle}</outer_angle>
-        <falloff>1</falloff>
-      </spot>
-      <direction>1 0 0</direction>
-    </light>
-  </xacro:macro>
 </robot>

Commit message: Fixed thruster macros

File: urdf/robots/polysat_description/urdf/polysat_base.xacro (robot description, xacro)
@@ -39,15 +39,15 @@
     <!-- Add thruster visuals -->
     <!-- Top -->
-    <!--<xacro:thruster_visual_macro namespace="$(arg namespace)" thruster_id="5" x="${-0.15/2}" y="${0.85}" z="0.5" R="0" P="0" Y="0"/>
+    <xacro:thruster_visual_macro namespace="$(arg namespace)" thruster_id="5" x="${-0.15/2}" y="${0.85}" z="0.5" R="0" P="0" Y="0"/>
     <xacro:thrust_plume_visual_macro namespace="$(arg namespace)" thruster_id="5" x="${-0.17}" y="${1.095}" z="0.55" R="${pi/2}" P="0" Y="0"/>
     <xacro:thruster_visual_macro namespace="$(arg namespace)" thruster_id="4" x="${-0.15/2}" y="${-1.0}" z="0.5" R="0" P="0" Y="0"/>
-    <xacro:thrust_plume_visual_macro namespace="$(arg namespace)" thruster_id="4" x="${-0.17}" y="${-0.755}" z="0.55" R="${pi/2}" P="0" Y="0"/-->
+    <xacro:thrust_plume_visual_macro namespace="$(arg namespace)" thruster_id="4" x="${-0.17}" y="${-0.755}" z="0.55" R="${pi/2}" P="0" Y="0"/>
     <!-- Bottom -->
-    <!--<xacro:thruster_visual_macro namespace="$(arg namespace)" thruster_id="6" x="${-0.15/2}" y="${1.0}" z="-0.5" R="${pi}" P="0" Y="0"/>
+    <xacro:thruster_visual_macro namespace="$(arg namespace)" thruster_id="6" x="${-0.15/2}" y="${1.0}" z="-0.5" R="${pi}" P="0" Y="0"/>
     <xacro:thrust_plume_visual_macro namespace="$(arg namespace)" thruster_id="6" x="${-0.17}" y="${0.755}" z="-0.55" R="${-pi/2}" P="0" Y="0"/>
     <xacro:thruster_visual_macro namespace="$(arg namespace)" thruster_id="7" x="${-0.15/2}" y="${-.85}" z="-0.5" R="${pi}" P="0" Y="0"/>
-    <xacro:thrust_plume_visual_macro namespace="$(arg namespace)" thruster_id="7" x="${-0.17}" y="${-1.095}" z="-0.55" R="${-pi/2}" P="0" Y="0"/-->
+    <xacro:thrust_plume_visual_macro namespace="$(arg namespace)" thruster_id="7" x="${-0.17}" y="${-1.095}" z="-0.55" R="${-pi/2}" P="0" Y="0"/>
     <!-- Front -->
-    <!--<xacro:thruster_visual_macro namespace="$(arg namespace)" thruster_id="8" x="${0.5}" y="${0.85}" z="${0.15/2}" R="0" P="${pi/2}" Y="0"/>
+    <xacro:thruster_visual_macro namespace="$(arg namespace)" thruster_id="8" x="${0.5}" y="${0.85}" z="${0.15/2}" R="0" P="${pi/2}" Y="0"/>
     <xacro:thrust_plume_visual_macro namespace="$(arg namespace)" thruster_id="8" x="${0.55}" y="${1.095}" z="-0.16" R="${0}" P="0" Y="${-pi/2}"/>
     <xacro:thruster_visual_macro namespace="$(arg namespace)" thruster_id="9" x="${0.5}" y="${-1.0}" z="${0.15/2}" R="${0}" P="${pi/2}" Y="0"/>
@@ -56,7 +56,7 @@
     <xacro:thrust_plume_visual_macro namespace="$(arg namespace)" thruster_id="1" x="${0.55}" y="${0.17}" z="-0.59" R="${0}" P="0" Y="${-pi/2}"/>
     <xacro:thruster_visual_macro namespace="$(arg namespace)" thruster_id="0" x="${0.5}" y="${-0.15/2}" z="0.5" R="${0}" P="${pi/2}" Y="0"/>
-    <xacro:thrust_plume_visual_macro namespace="$(arg namespace)" thruster_id="0" x="${0.55}" y="${0.17}" z="0.26" R="${0}" P="0" Y="${-pi/2}"/-->
+    <xacro:thrust_plume_visual_macro namespace="$(arg namespace)" thruster_id="0" x="${0.55}" y="${0.17}" z="0.26" R="${0}" P="0" Y="${-pi/2}"/>
     <!-- Back -->
-    <!--<xacro:thruster_visual_macro namespace="$(arg namespace)" thruster_id="10" x="${-0.5}" y="${0.85}" z="${-0.15/2}" R="0" P="${-pi/2}" Y="0"/>
+    <xacro:thruster_visual_macro namespace="$(arg namespace)" thruster_id="10" x="${-0.5}" y="${0.85}" z="${-0.15/2}" R="0" P="${-pi/2}" Y="0"/>
     <xacro:thrust_plume_visual_macro namespace="$(arg namespace)" thruster_id="10" x="${-0.55}" y="${0.76}" z="-0.16" R="${0}" P="0" Y="${pi/2}"/>
     <xacro:thruster_visual_macro namespace="$(arg namespace)" thruster_id="11" x="${-0.5}" y="${-1.0}" z="${-0.15/2}" R="${0}" P="${-pi/2}" Y="0"/>
@@ -65,10 +65,10 @@
     <xacro:thrust_plume_visual_macro namespace="$(arg namespace)" thruster_id="3" x="${-0.55}" y="${-0.17}" z="-0.59" R="${0}" P="0" Y="${pi/2}"/>
     <xacro:thruster_visual_macro namespace="$(arg namespace)" thruster_id="2" x="${-0.5}" y="${-0.15/2}" z="0.35" R="${0}" P="${-pi/2}" Y="0"/>
-    <xacro:thrust_plume_visual_macro namespace="$(arg namespace)" thruster_id="2" x="${-0.55}" y="${-0.17}" z="0.26" R="${0}" P="0" Y="${pi/2}"/-->
+    <xacro:thrust_plume_visual_macro namespace="$(arg namespace)" thruster_id="2" x="${-0.55}" y="${-0.17}" z="0.26" R="${0}" P="0" Y="${pi/2}"/>
     <!-- Sides -->
-    <!--<xacro:thruster_visual_macro namespace="$(arg namespace)" thruster_id="12" x="${-0.15/2}" y="${-1.0}" z="${-0.15/2}" R="${pi/2}" P="${0}" Y="0"/>
+    <xacro:thruster_visual_macro namespace="$(arg namespace)" thruster_id="12" x="${-0.15/2}" y="${-1.0}" z="${-0.15/2}" R="${pi/2}" P="${0}" Y="0"/>
     <xacro:thrust_plume_visual_macro namespace="$(arg namespace)" thruster_id="12" x="${0.17}" y="${-1.05}" z="-0.17" R="${0}" P="0" Y="${pi}"/>
     <xacro:thruster_visual_macro namespace="$(arg namespace)" thruster_id="13" x="${-0.15/2}" y="${1.0}" z="${0.15/2}" R="${-pi/2}" P="${0}" Y="${0}"/>
-    <xacro:thrust_plume_visual_macro namespace="$(arg namespace)" thruster_id="13" x="${0.17}" y="${1.05}" z="0.17" R="${0}" P="${pi}" Y="${0}"/-->
+    <xacro:thrust_plume_visual_macro namespace="$(arg namespace)" thruster_id="13" x="${0.17}" y="${1.05}" z="0.17" R="${0}" P="${pi}" Y="${0}"/>
     <!-- Add maneuvering thrusters -->
     <xacro:thruster_macro namespace="${namespace}" thruster_id="0">

File: urdf/robots/polysat_description/urdf/polysat_thrusters.xacro (robot description, xacro)
@@ -3,11 +3,7 @@
   <xacro:macro name="thruster_macro" params="namespace thruster_id *origin">
     <link name="${namespace}/thruster_${thruster_id}">
-      <inertial>
+      <xacro:box_inertial x="0.001" y="0.001" z="0.001" mass="0.0001">
         <origin xyz="0 0 0" rpy="0 0 0"/>
-        <mass value="0.001"/>
-        <inertia ixx="0.001" ixy="0.0" ixz="0.0"
-                 iyy="0.001" iyz="0.0"
-                 izz="0.001"/>
-      </inertial>
+      </xacro:box_inertial>
       <visual>
         <geometry>
@@ -45,3 +41,12 @@
     </gazebo>
   </xacro:macro>
+  <xacro:macro name="box_inertial" params="x y z mass *origin">
+    <inertial>
+      <mass value="${mass}"/>
+      <xacro:insert_block name="origin"/>
+      <inertia ixx="0.00001" ixy="0.0" ixz="0.0"
+               iyy="0.00001" iyz="0.0"
+               izz="0.00001"/>
+    </inertial>
+  </xacro:macro>
 </robot>
