Commit message: Added hokuyo_lx30, yet to test

File: urdf/robots/polysat_description/urdf/polysat_base.xacro (robot description, xacro)
@@ -119,5 +119,5 @@
     </gazebo>
     <xacro:arg name="inertial_reference_frame" default="world"/>
-    <xacro:include filename="$(find sc_gazebo_plugins)/urdf/imu.xacro"/>
+    <!--xacro:include filename="$(find sc_gazebo_plugins)/urdf/imu.xacro"/>
     <xacro:default_imu_macro
       namespace="$(arg namespace)"
@@ -130,5 +130,5 @@
       namespace="$(arg namespace)"
       parent_link="$(arg namespace)/base_link">
-    </xacro:default_pose_3d>
+    </xacro:default_pose_3d-->
    </xacro:macro>
 </robot>

File: urdf/robots/polysat_description/urdf/polysat_robot.urdf.xacro (robot description, xacro)
@@ -8,5 +8,6 @@
   <xacro:include filename="$(find polysat_description)/urdf/polysat_base.xacro"/>
   <xacro:polysat_base namespace="$(arg namespace)"/>
-  <!--xacro:include filename="$(find polysat_description)/urdf/polysat_sensors.xacro"/-->
+  <xacro:include filename="$(find polysat_description)/urdf/polysat_sensors.xacro"/>
+  <xacro:add_sensors namespace="$(arg namespace)" inertial_reference_frame="$(arg inertial_reference_frame)"/>
   <!-- oberon7 -->
   <xacro:include filename="$(find oberon7_description)/urdf/oberon7.urdf.xacro"/>

File: urdf/robots/polysat_description/urdf/polysat_sensors.xacro (robot description, xacro)
@@ -3,15 +3,23 @@
   <xacro:include filename="$(find sc_gazebo_plugins)/urdf/imu.xacro"/>
   <xacro:include filename="$(find sc_gazebo_plugins)/urdf/pose_3d.xacro"/>
-  <!-- IMU  -->
-  <xacro:default_imu_macro
-    namespace="${namespace}"
-    parent_link="${namespace}/base_link"
-    inertial_reference_frame="${inertial_reference_frame}">
-    <origin xyz="0 0 0" rpy="0 0 0"/>
-  </xacro:default_imu_macro>
-  <!-- GT Pose -->
-  <xacro:default_pose_3d
-    namespace="${namespace}"
-    parent_link="${namespace}/base_link">
-  </xacro:default_pose_3d>
+  <xacro:include filename="$(find sc_gazebo_plugins)/urdf/hokuyo_lx30.xacro"/>
+  <xacro:macro name="add_sensors" params="namespace inertial_reference_frame">
+    <!-- IMU  -->
+    <xacro:default_imu_macro
+      namespace="${namespace}"
+      parent_link="${namespace}/base_link"
+      inertial_reference_frame="${inertial_reference_frame}">
+      <origin xyz="0 0 0" rpy="0 0 0"/>
+    </xacro:default_imu_macro>
+    <!-- GT Pose -->
+    <xacro:default_pose_3d
+      namespace="${namespace}"
+      parent_link="${namespace}/base_link">
+    </xacro:default_pose_3d>
+    <!-- hokuyo node -->
+    <xacro:hokuyo_macro
+      namespace="${namespace}"
+      parent_link="${namespace}/base_link">
+    </xacro:hokuyo_macro>
+  </xacro:macro>
 </robot>

Commit message: Added tf broadcaster

File: urdf/robots/polysat_description/urdf/polysat_base.xacro (robot description, xacro)
@@ -119,16 +119,3 @@
     </gazebo>
     <xacro:arg name="inertial_reference_frame" default="world"/>
-    <!--xacro:include filename="$(find sc_gazebo_plugins)/urdf/imu.xacro"/>
-    <xacro:default_imu_macro
-      namespace="$(arg namespace)"
-      parent_link="$(arg namespace)/base_link"
-      inertial_reference_frame="$(arg inertial_reference_frame)">
-      <origin xyz="0 0 0" rpy="0 0 0"/>
-    </xacro:default_imu_macro>
-    <xacro:include filename="$(find sc_gazebo_plugins)/urdf/pose_3d.xacro"/>
-    <xacro:default_pose_3d
-      namespace="$(arg namespace)"
-      parent_link="$(arg namespace)/base_link">
-    </xacro:default_pose_3d-->
-   </xacro:macro>
 </robot>

Commit message: Fixed bug in polysat_base

File: urdf/robots/polysat_description/urdf/polysat_base.xacro (robot description, xacro)
@@ -119,3 +119,4 @@
     </gazebo>
     <xacro:arg name="inertial_reference_frame" default="world"/>
+  </xacro:macro>
 </robot>

Commit message: Cube with color imported

File: urdf/robots/polysat_description/urdf/polysat_base.xacro (robot description, xacro)
@@ -21,5 +21,5 @@
         <origin xyz="-0.5 1.0 -0.5" rpy="1.570796326794 0 0"/>
         <geometry>
-          <mesh filename="file://$(find polysat_description)/meshes/base.stl" scale="0.001 0.001 0.001"/>
+          <mesh filename="file://$(find sc_models)/models/import_cube/untitled.dae" scale="1 1 1"/>
         </geometry>
       </visual>
@@ -27,5 +27,5 @@
         <origin xyz="-0.5 1.0 -0.5" rpy="1.570796326794 0 0"/>
         <geometry>
-          <mesh filename="file://$(find polysat_description)/meshes/base.stl" scale="0.001 0.001 0.001"/>
+          <mesh filename="file://$(find sc_models)/models/import_cube/untitled.dae" scale="1 1 1"/>
         </geometry>
       </collision>

Commit message: Corrected polysat model

File: urdf/robots/polysat_description/urdf/polysat_base.xacro (robot description, xacro)
@@ -22,5 +22,5 @@
         <origin xyz="-0.5 1.0 -0.5" rpy="1.570796326794 0 0"/>
         <geometry>
-          <mesh filename="file://$(find sc_models)/models/import_cube/untitled.dae" scale="1 1 1"/>
+          <mesh filename="file://$(find polysat_description)/meshes/base.stl" scale="0.001 0.001 0.001"/>
         </geometry>
       </visual>
@@ -28,5 +28,5 @@
         <origin xyz="-0.5 1.0 -0.5" rpy="1.570796326794 0 0"/>
         <geometry>
-          <mesh filename="file://$(find sc_models)/models/import_cube/untitled.dae" scale="1 1 1"/>
+          <mesh filename="file://$(find polysat_description)/meshes/base.stl" scale="0.001 0.001 0.001"/>
         </geometry>
       </collision>

Commit message: Added camera plugin xacro file from uuv simulator, tested on polysat

File: urdf/robots/polysat_description/urdf/polysat_base.xacro (robot description, xacro)
@@ -6,4 +6,5 @@
   <xacro:include filename="$(find polysat_description)/urdf/polysat_thrusters.xacro"/>
   <xacro:include filename="$(find polysat_description)/urdf/polysat_thruster_visuals.xacro"/>
+  <xacro:include filename="$(find sc_gazebo_plugins)/urdf/camera.xacro"/>
   <xacro:macro name="polysat_base" params="namespace">
     <!-- "Dummy base link to eliminate root link inertia warning -->
@@ -38,4 +39,19 @@
       <child link="$(arg namespace)/polysat_link"/>
     </joint>
+    <!-- Add camera -->
+    <xacro:regular_camera_plugin_macro namespace="$(arg namespace)"
+      suffix="1"
+      parent_link="$(arg namespace)/polysat_link"
+      topic="camera_topic"
+      mass="0.01"
+      update_rate="30"
+      hfov="1.5125"
+      width="640"
+      height="480"
+      stddev="0.02"
+      scale="1.0">
+      <origin xyz="0 0 2" rpy="0 0 0"/>
+      <inertia ixx="0.00001" ixy="0.0" ixz="0.0" iyy="0.00001" iyz="0.0" izz="0.000001"/>
+    </xacro:regular_camera_plugin_macro>
     <!-- Add thruster visuals -->
     <!-- Top -->

Commit message: blargh

File: urdf/robots/polysat_description/urdf/polysat_base.xacro (robot description, xacro)
@@ -135,5 +135,5 @@
       </plugin>
     </gazebo>
-    <xacro:arg name="inertial_reference_frame" default="world"/>
+    <!--xacro:arg name="inertial_reference_frame" default="world"/-->
   </xacro:macro>
 </robot>

File: urdf/robots/prime_description/urdf/prime_base.xacro (robot description, xacro)
@@ -11,7 +11,7 @@
         <mass value="13.0"/>
         <inertia
-          ixx="30.0" ixy="0.0" ixz="0.0"
-          iyy="30.0" iyz="0.0"
-          izz="20.0"/>
+          ixx="0.15795" ixy="0.0" ixz="0.0"
+          iyy="0.15795" iyz="0.0"
+          izz="0.15795"/>
       </inertial>
       <visual>
@@ -46,7 +46,7 @@
         <mass value="0.5"/>
         <inertia
-          ixx="0.5" ixy="0.0" ixz="0.0"
-          iyy="0.5" iyz="0.0"
-          izz="0.25"/>
+          ixx="0.0416833" ixy="0.0" ixz="0.0"
+          iyy="0.0000333" iyz="0.0"
+          izz="0.0416833"/>
       </inertial>
       <visual>
@@ -74,5 +74,5 @@
         <torsion_joint>${namespace}/torsion_spring_joint</torsion_joint>
         <kx>0.11</kx>
-        <set_point>0.05</set_point>
+        <set_point>0.0</set_point>
       </plugin>
     </gazebo>

File: urdf/robots/prime_description/urdf/prime_robot.urdf.xacro (robot description, xacro)
@@ -8,4 +8,16 @@
   <xacro:include filename="$(find prime_description)/urdf/prime_base.xacro"/>
   <xacro:prime_base namespace="$(arg namespace)"/>
+  <xacro:include filename="$(find sc_gazebo_plugins)/urdf/imu.xacro"/>
+  <xacro:default_imu_macro
+    namespace="$(arg namespace)"
+    parent_link="$(arg namespace)/base_link"
+    inertial_reference_frame="$(arg inertial_reference_frame)">
+    <origin xyz="0 0 0" rpy="0 0 0"/>
+  </xacro:default_imu_macro>
+  <xacro:include filename="$(find sc_gazebo_plugins)/urdf/pose_3d.xacro"/>
+  <xacro:default_pose_3d
+    namespace="$(arg namespace)"
+    parent_link="$(arg namespace)/base_link">
+  </xacro:default_pose_3d>
   <!--xacro:include filename="$(find prime_description)/urdf/prime_reaction_wheels.xacro"/>
   <xacro:add_wheels namespace="$(arg namespace)"/-->
