Commit message: Re-oriented all thruster visuals

File: urdf/robots/polysat_perseus_description/urdf/polysat_base.xacro (robot description, xacro)
@@ -20,13 +20,13 @@
       </inertial>
       <visual>
-        <origin xyz="${sf*-0.5} ${sf*1.0} ${sf*-0.5}" rpy="1.570796326794 0 0"/>
+        <origin xyz="${sf*0} ${sf*0} ${sf*0}" rpy="0 0 0"/>
         <geometry>
-          <mesh filename="file://$(find polysat_description)/meshes/base.stl" scale="${sf*0.001} ${sf*0.001} ${sf*0.001}"/>
+          <box size="${sf*2} ${sf*1} ${sf*1}"/>
         </geometry>
       </visual>
       <collision>
-        <origin xyz="${sf*-0.5} ${sf*1.0} ${sf*-0.5}" rpy="1.570796326794 0 0"/>
+        <origin xyz="${sf*0} ${sf*0} ${sf*0}" rpy="0 0 0"/>
         <geometry>
-          <mesh filename="file://$(find polysat_description)/meshes/base.stl" scale="${sf*0.001} ${sf*0.001} ${sf*0.001}"/>
+          <box size="${sf*2} ${sf*1} ${sf*1}"/>
         </geometry>
       </collision>
@@ -40,36 +40,36 @@
     <!-- Add thruster visuals -->
     <!-- Top -->
-    <xacro:thruster_visual_macro namespace="$(arg namespace)" thruster_id="5" sfac="${sf}" x="${sf*-0.15/2}" y="${sf*0.85}" z="${sf*0.5}" R="0" P="0" Y="0"/>
-    <xacro:thrust_plume_visual_macro namespace="$(arg namespace)" thruster_id="6" sfac="${sf}" x="${sf*-0.17}" y="${sf*1.095}" z="${sf*0.55}" R="${pi/2}" P="0" Y="0"/>
-    <xacro:thruster_visual_macro namespace="$(arg namespace)" thruster_id="4" sfac="${sf}" x="${sf*-0.15/2}" y="${sf*-1.0}" z="${sf*0.5}" R="0" P="0" Y="0"/>
-    <xacro:thrust_plume_visual_macro namespace="$(arg namespace)" thruster_id="7" sfac="${sf}" x="${sf*-0.17}" y="${sf*-0.755}" z="${sf*0.55}" R="${pi/2}" P="0" Y="0"/>
+    <xacro:thruster_visual_macro namespace="$(arg namespace)" thruster_id="5" sfac="${sf}" x="${sf*-0.075}" y="${sf*(0.5-0.15)}" z="${sf*0.5}" R="0" P="0" Y="0"/>
+    <xacro:thruster_visual_macro namespace="$(arg namespace)" thruster_id="4" sfac="${sf}" x="${sf*-0.075}" y="${sf*-0.5}" z="${sf*0.5}" R="0" P="0" Y="0"/>
+    <xacro:thrust_plume_visual_macro namespace="$(arg namespace)" thruster_id="6" sfac="${sf}" x="${sf*-0.17}" y="${sf*0.595}" z="${sf*0.55}" R="${pi/2}" P="0" Y="0"/>
+    <xacro:thrust_plume_visual_macro namespace="$(arg namespace)" thruster_id="7" sfac="${sf}" x="${sf*-0.17}" y="${sf*-0.255}" z="${sf*0.55}" R="${pi/2}" P="0" Y="0"/>
     <!-- Bottom -->
-    <xacro:thruster_visual_macro namespace="$(arg namespace)" thruster_id="6" sfac="${sf}" x="${sf*-0.15/2}" y="${sf*1.0}" z="${sf*-0.5}" R="${pi}" P="0" Y="0"/>
-    <xacro:thrust_plume_visual_macro namespace="$(arg namespace)" thruster_id="5" sfac="${sf}" x="${sf*-0.17}" y="${sf*0.755}" z="${sf*-0.55}" R="${-pi/2}" P="0" Y="0"/>
-    <xacro:thruster_visual_macro namespace="$(arg namespace)" thruster_id="7" sfac="${sf}" x="${sf*-0.15/2}" y="${sf*-.85}" z="${sf*-0.5}" R="${pi}" P="0" Y="0"/>
-    <xacro:thrust_plume_visual_macro namespace="$(arg namespace)" thruster_id="4" sfac="${sf}" x="${sf*-0.17}" y="${sf*-1.095}" z="${sf*-0.55}" R="${-pi/2}" P="0" Y="0"/>
+    <xacro:thruster_visual_macro namespace="$(arg namespace)" thruster_id="6" sfac="${sf}" x="${sf*-0.15/2}" y="${sf*0.5}" z="${sf*-0.5}" R="${pi}" P="0" Y="0"/>
+    <xacro:thruster_visual_macro namespace="$(arg namespace)" thruster_id="7" sfac="${sf}" x="${sf*-0.15/2}" y="${sf*(-0.5+0.15)}" z="${sf*-0.5}" R="${pi}" P="0" Y="0"/>
+    <xacro:thrust_plume_visual_macro namespace="$(arg namespace)" thruster_id="5" sfac="${sf}" x="${sf*-0.17}" y="${sf*0.255}" z="${sf*-0.55}" R="${-pi/2}" P="0" Y="0"/>
+    <xacro:thrust_plume_visual_macro namespace="$(arg namespace)" thruster_id="4" sfac="${sf}" x="${sf*-0.17}" y="${sf*-0.595}" z="${sf*-0.55}" R="${-pi/2}" P="0" Y="0"/>
     <!-- Front -->
-    <xacro:thruster_visual_macro namespace="$(arg namespace)" thruster_id="8" sfac="${sf}" x="${sf*0.5}" y="${sf*0.85}" z="${sf*.15/2}" R="0" P="${pi/2}" Y="0"/>
-    <xacro:thrust_plume_visual_macro namespace="$(arg namespace)" thruster_id="10" sfac="${sf}" x="${sf*0.55}" y="${sf*1.095}" z="${sf*-0.16}" R="${0}" P="0" Y="${-pi/2}"/>
-    <xacro:thruster_visual_macro namespace="$(arg namespace)" thruster_id="9" sfac="${sf}" x="${sf*0.5}" y="${sf*-1.0}" z="${sf*0.15/2}" R="${0}" P="${pi/2}" Y="0"/>
-    <xacro:thrust_plume_visual_macro namespace="$(arg namespace)" thruster_id="11" sfac="${sf}" x="${sf*0.55}" y="${sf*-0.76}" z="${sf*-0.17}" R="${0}" P="0" Y="${-pi/2}"/>
-    <xacro:thruster_visual_macro namespace="$(arg namespace)" thruster_id="1" sfac="${sf}" x="${sf*0.5}" y="${sf*-0.15/2}" z="${sf*-0.35}" R="${0}" P="${pi/2}" Y="0"/>
-    <xacro:thrust_plume_visual_macro namespace="$(arg namespace)" thruster_id="3" sfac="${sf}" x="${sf*0.55}" y="${sf*0.17}" z="${sf*-0.59}" R="${0}" P="0" Y="${-pi/2}"/>
-    <xacro:thruster_visual_macro namespace="$(arg namespace)" thruster_id="0" sfac="${sf}" x="${sf*0.5}" y="${sf*-0.15/2}" z="${sf*0.5}" R="${0}" P="${pi/2}" Y="0"/>
-    <xacro:thrust_plume_visual_macro namespace="$(arg namespace)" thruster_id="2" sfac="${sf}" x="${sf*0.55}" y="${sf*0.17}" z="${sf*0.26}" R="${0}" P="0" Y="${-pi/2}"/>
+    <xacro:thruster_visual_macro namespace="$(arg namespace)" thruster_id="8" sfac="${sf}" x="${sf*1}" y="${sf*(0.5-0.15)}" z="${sf*(0+0.075)}" R="0" P="${pi/2}" Y="0"/>
+    <xacro:thruster_visual_macro namespace="$(arg namespace)" thruster_id="9" sfac="${sf}" x="${sf*1}" y="${sf*-0.5}" z="${sf*(0+0.075)}" R="${0}" P="${pi/2}" Y="0"/>
+    <xacro:thruster_visual_macro namespace="$(arg namespace)" thruster_id="1" sfac="${sf}" x="${sf*1}" y="${sf*-0.15/2}" z="${sf*(-0.5+0.15)}" R="${0}" P="${pi/2}" Y="0"/>
+    <xacro:thruster_visual_macro namespace="$(arg namespace)" thruster_id="0" sfac="${sf}" x="${sf*1}" y="${sf*-0.15/2}" z="${sf*0.5}" R="${0}" P="${pi/2}" Y="0"/>
+    <xacro:thrust_plume_visual_macro namespace="$(arg namespace)" thruster_id="10" sfac="${sf}" x="${sf*1.05}" y="${sf*0.595}" z="${sf*-0.16}" R="${0}" P="0" Y="${-pi/2}"/>
+    <xacro:thrust_plume_visual_macro namespace="$(arg namespace)" thruster_id="11" sfac="${sf}" x="${sf*1.05}" y="${sf*-0.26}" z="${sf*-0.17}" R="${0}" P="0" Y="${-pi/2}"/>
+    <xacro:thrust_plume_visual_macro namespace="$(arg namespace)" thruster_id="3" sfac="${sf}" x="${sf*1.05}" y="${sf*0.17}" z="${sf*-0.59}" R="${0}" P="0" Y="${-pi/2}"/>
+    <xacro:thrust_plume_visual_macro namespace="$(arg namespace)" thruster_id="2" sfac="${sf}" x="${sf*1.05}" y="${sf*0.17}" z="${sf*0.26}" R="${0}" P="0" Y="${-pi/2}"/>
     <!-- Back -->
-    <xacro:thruster_visual_macro namespace="$(arg namespace)" thruster_id="10" sfac="${sf}" x="${sf*-0.5}" y="${sf*0.85}" z="${sf*-0.15/2}" R="0" P="${-pi/2}" Y="0"/>
-    <xacro:thrust_plume_visual_macro namespace="$(arg namespace)" thruster_id="8" sfac="${sf}" x="${sf*-0.55}" y="${sf*0.76}" z="${sf*-0.16}" R="${0}" P="0" Y="${pi/2}"/>
-    <xacro:thruster_visual_macro namespace="$(arg namespace)" thruster_id="11" sfac="${sf}" x="${sf*-0.5}" y="${sf*-1.0}" z="${sf*-0.15/2}" R="${0}" P="${-pi/2}" Y="0"/>
-    <xacro:thrust_plume_visual_macro namespace="$(arg namespace)" thruster_id="9" sfac="${sf}" x="${sf*-0.55}" y="${sf*-1.095}" z="${sf*-0.17}" R="${0}" P="0" Y="${pi/2}"/>
-    <xacro:thruster_visual_macro namespace="$(arg namespace)" thruster_id="3" sfac="${sf}" x="${sf*-0.5}" y="${sf*-0.15/2}" z="${sf*-0.5}" R="${0}" P="${-pi/2}" Y="0"/>
-    <xacro:thrust_plume_visual_macro namespace="$(arg namespace)" thruster_id="1" sfac="${sf}" x="${sf*-0.55}" y="${sf*-0.17}" z="${sf*-0.59}" R="${0}" P="0" Y="${pi/2}"/>
-    <xacro:thruster_visual_macro namespace="$(arg namespace)" thruster_id="2" sfac="${sf}" x="${sf*-0.5}" y="${sf*-0.15/2}" z="${sf*0.35}" R="${0}" P="${-pi/2}" Y="0"/>
-    <xacro:thrust_plume_visual_macro namespace="$(arg namespace)" thruster_id="0" sfac="${sf}" x="${sf*-0.55}" y="${sf*-0.17}" z="${sf*0.26}" R="${0}" P="0" Y="${pi/2}"/>
+    <xacro:thruster_visual_macro namespace="$(arg namespace)" thruster_id="10" sfac="${sf}" x="${sf*-1}" y="${sf*(0.5-0.15)}" z="${sf*(0-0.075)}" R="0" P="${-pi/2}" Y="0"/>
+    <xacro:thruster_visual_macro namespace="$(arg namespace)" thruster_id="11" sfac="${sf}" x="${sf*-1}" y="${sf*-0.5}" z="${sf*(0-0.075)}" R="${0}" P="${-pi/2}" Y="0"/>
+    <xacro:thruster_visual_macro namespace="$(arg namespace)" thruster_id="3" sfac="${sf}" x="${sf*-1}" y="${sf*(0-0.075)}" z="${sf*-0.5}" R="${0}" P="${-pi/2}" Y="0"/>
+    <xacro:thruster_visual_macro namespace="$(arg namespace)" thruster_id="2" sfac="${sf}" x="${sf*-1}" y="${sf*(0-0.075)}" z="${sf*(0.5-0.15)}" R="${0}" P="${-pi/2}" Y="0"/>
+    <xacro:thrust_plume_visual_macro namespace="$(arg namespace)" thruster_id="8" sfac="${sf}" x="${sf*-1.05}" y="${sf*0.26}" z="${sf*-0.16}" R="${0}" P="0" Y="${pi/2}"/>
+    <xacro:thrust_plume_visual_macro namespace="$(arg namespace)" thruster_id="9" sfac="${sf}" x="${sf*-1.05}" y="${sf*-0.595}" z="${sf*-0.17}" R="${0}" P="0" Y="${pi/2}"/>
+    <xacro:thrust_plume_visual_macro namespace="$(arg namespace)" thruster_id="1" sfac="${sf}" x="${sf*-1.05}" y="${sf*-0.17}" z="${sf*-0.59}" R="${0}" P="0" Y="${pi/2}"/>
+    <xacro:thrust_plume_visual_macro namespace="$(arg namespace)" thruster_id="0" sfac="${sf}" x="${sf*-1.05}" y="${sf*-0.17}" z="${sf*0.26}" R="${0}" P="0" Y="${pi/2}"/>
     <!-- Sides -->
-    <xacro:thruster_visual_macro namespace="$(arg namespace)" thruster_id="12" sfac="${sf}" x="${sf*-0.15/2}" y="${sf*-1.0}" z="${sf*-0.15/2}" R="${pi/2}" P="${0}" Y="0"/>
-    <xacro:thrust_plume_visual_macro namespace="$(arg namespace)" thruster_id="12" sfac="${sf}" x="${sf*0.17}" y="${sf*-1.05}" z="${sf*-0.17}" R="${0}" P="0" Y="${pi}"/>
-    <xacro:thruster_visual_macro namespace="$(arg namespace)" thruster_id="13" sfac="${sf}" x="${sf*-0.15/2}" y="${sf*1.0}" z="${sf*0.15/2}" R="${-pi/2}" P="${0}" Y="${0}"/>
-    <xacro:thrust_plume_visual_macro namespace="$(arg namespace)" thruster_id="13" sfac="${sf}" x="${sf*0.17}" y="${sf*1.05}" z="${sf*0.17}" R="${0}" P="${pi}" Y="${0}"/>
+    <xacro:thruster_visual_macro namespace="$(arg namespace)" thruster_id="12" sfac="${sf}" x="${sf*-0.15/2}" y="${sf*-0.5}" z="${sf*-0.15/2}" R="${pi/2}" P="${0}" Y="0"/>
+    <xacro:thruster_visual_macro namespace="$(arg namespace)" thruster_id="13" sfac="${sf}" x="${sf*-0.15/2}" y="${sf*0.5}" z="${sf*0.15/2}" R="${-pi/2}" P="${0}" Y="${0}"/>
+    <xacro:thrust_plume_visual_macro namespace="$(arg namespace)" thruster_id="12" sfac="${sf}" x="${sf*0.17}" y="${sf*-0.55}" z="${sf*-0.17}" R="${0}" P="0" Y="${pi}"/>
+    <xacro:thrust_plume_visual_macro namespace="$(arg namespace)" thruster_id="13" sfac="${sf}" x="${sf*0.17}" y="${sf*0.55}" z="${sf*0.17}" R="${0}" P="${pi}" Y="${0}"/>
     <!-- Add maneuvering thrusters -->
     <xacro:thruster_macro namespace="${namespace}" thruster_id="0">

File: urdf/robots/polysat_perseus_description/urdf/polysat_robot.urdf.xacro (robot description, xacro)
@@ -21,10 +21,10 @@
     <parent link="$(arg namespace)/base_link"/>
     <child link="perseus_l/base"/>
-    <origin rpy="0 -1.57079632 0" xyz="0.10 0.32 -0.00"/>
+    <origin rpy="0 -3.14159265 0" xyz="0.25 0.15 -0.00"/>
   </joint>
   <joint name="perseus_r_anchor" type="fixed">
     <parent link="$(arg namespace)/base_link"/>
     <child link="perseus_r/base"/>
-    <origin rpy="3.14159265 1.57079632 0" xyz="0.10 -0.32 -0.00"/>
+    <origin rpy="3.14159265 3.14159265 0" xyz="0.25 -0.15 -0.00"/>
   </joint>
 </robot>
