Commit message: Added a cubesat description, tested basic reaction wheel plugin. Check AddTorque vs AddRelativeTorque

File: sc_gazebo_plugins/urdf/reaction_wheel.xacro (robot description, xacro)
@@ -4,8 +4,8 @@
     <link name="${namespace}/wheel_${wheel_id}_link">
       <inertial>
-        <mass value="0.1"/>
-        <inertia ixx="0.00001" ixy="0.0" ixz="0.0"
-                 iyy="0.00001" iyz="0.0"
-                 izz="0.00001"/>
+        <mass value="10"/>
+        <inertia ixx="1" ixy="0.0" ixz="0.0"
+                 iyy="1" iyz="0.0"
+                 izz="1"/>
       </inertial>
       <visual>
@@ -16,22 +16,22 @@
       </visual>
       <collision>
-        <geomtery>
+        <geometry>
           <cylinder length="0.0000001" radius="0.0000001"/>
         </geometry>
       </collision>
     </link>
-    <joint name="${namespace}/wheel_${wheel_id}_joint" type="fixed">
+    <joint name="${namespace}/wheel_${wheel_id}_joint" type="revolute">
       <xacro:insert_block name="origin"/>
       <parent link="${namespace}/base_link"/>
       <child link="${namespace}/wheel_${wheel_id}_link"/>
-      <axis xyz="1 0 0"/>
+      <limit effort="0" lower="0" upper="0" velocity="0"/>
     </joint>
     <gazebo>
       <plugin name="${namespace}_${wheel_id}_reaction_wheel_model" filename="libsc_reaction_wheel_plugin.so">
-        <wheel>
-          <linkName>${namespace}/wheel_${wheel_id}_link</linkName>
+        <reaction_wheel>
+          <linkName>${namespace}/base_link</linkName>
           <jointName>${namespace}/wheel_${wheel_id}_joint</jointName>
           <cmdTopic>${namespace}/wheels/wheel_${wheel_id}</cmdTopic>
-        </wheel>
+        </reaction_wheel>
       </plugin>
     </gazebo>

File: urdf/robots/polysat_description/urdf/polysat_base.xacro (robot description, xacro)
@@ -3,4 +3,5 @@
   <!-- <xacro:property name="debug" default="false"/> -->
   <xacro:arg name="namespace" default="polysat"/>
+  <xacro:include filename="$(find sc_gazebo_plugins)/urdf/reaction_wheel.xacro"/>
   <xacro:include filename="$(find polysat_description)/urdf/polysat_thrusters.xacro"/>
   <xacro:include filename="$(find polysat_description)/urdf/polysat_thruster_visuals.xacro"/>

Commit message: Tested prime on table, next add spring to experiment setup and test

File: sc_gazebo_plugins/urdf/reaction_wheel.xacro (robot description, xacro)
@@ -4,5 +4,5 @@
     <link name="${namespace}/wheel_${wheel_id}_link">
       <inertial>
-        <mass value="10"/>
+        <mass value="1"/>
         <inertia ixx="1" ixy="0.0" ixz="0.0"
                  iyy="1" iyz="0.0"

File: urdf/robots/cubesat_description/urdf/cubesat_base.xacro (robot description, xacro)
@@ -1,5 +1,4 @@
 <?xml version="1.0"?>
 <robot name="cubesat" xmlns:xacro="https://www.ros.org/wiki/xacro">
-  <!-- <xacro:property name="debug" default="false"/> -->
   <xacro:arg name="namespace" default="cubesat"/>
   <xacro:macro name="cubesat_base" params="namespace">
