Commit message: Solved apriltag_ros usage issue

File: sc_gazebo_plugins/urdf/camera.xacro (robot description, xacro)
@@ -5,5 +5,5 @@
             width height stddev scale *inertia *origin">
     <!-- Sensor link -->
-    <link name="${namespace}/camera${suffix}_link">
+    <link name="${namespace}/camera_link">
       <inertial>
         <origin xyz="0 0 0" rpy="0 0 0"/>
@@ -21,12 +21,12 @@
       <xacro:no_collision/>
     </link>
-    <joint name="${namespace}/camer${suffix}_joint" type="revolute">
+    <joint name="${namespace}/camer_joint" type="revolute">
       <xacro:insert_block name="origin"/>
       <parent link="${parent_link}"/>
-      <child link="${namespace}/camera${suffix}_link"/>
+      <child link="${namespace}/camera_link"/>
       <limit upper="0" lower="0" effort="0" velocity="0"/>
       <axis xyz="1 0 0"/>
     </joint>
-    <link name="${namespace}/camera${suffix}_link_optical">
+    <link name="${namespace}/camera_link_optical">
       <inertial>
         <origin xyz="0 0 0" rpy="0 0 0"/>
@@ -44,15 +44,15 @@
       </collision>
     </link>
-    <joint name="${namespace}/camera${suffix}_optical_joint" type="revolute">
+    <joint name="${namespace}/camera_optical_joint" type="revolute">
       <origin xyz="0 0 0" rpy="${-pi/2} 0 ${-pi/2}"/>
-      <parent link="${namespace}/camera${suffix}_link"/>
-      <child link="${namespace}/camera${suffix}_link_optical"/>
+      <parent link="${namespace}/camera_link"/>
+      <child link="${namespace}/camera_link_optical"/>
       <limit upper="0" lower="0" effort="0" velocity="0"/>
       <axis xyz="1 0 0"/>
     </joint>
-    <gazebo reference="${namespace}/camera${suffix}_link">
-      <sensor type="camera" name="camera${suffix}">
+    <gazebo reference="${namespace}/camera_link">
+      <sensor type="camera" name="camera">
         <update_rate>${update_rate}</update_rate>
-        <camera name="camera${suffix}">
+        <camera name="camera">
           <horizontal_fov>${hfov}</horizontal_fov>
           <image>
@@ -71,8 +71,8 @@
           </noise>
         </camera>
-        <plugin name="camera${suffix}_controller" filename="libgazebo_ros_camera.so">
+        <plugin name="camera_controller" filename="libgazebo_ros_camera.so">
           <updateRate>${update_rate}</updateRate>
-          <cameraName>${namespace}/camera${suffix}</cameraName>
-          <frameName>camera${suffix}_link_optical</frameName>
+          <cameraName>camera</cameraName>
+          <frameName>camera_link_optical</frameName>
           <attenuationR>0.0</attenuationR>
           <attenuationG>0.0</attenuationG>

File: urdf/robots/polysat_description/urdf/polysat_base.xacro (robot description, xacro)
@@ -43,5 +43,5 @@
       suffix="1"
       parent_link="$(arg namespace)/polysat_link"
-      topic="image_rect"
+      topic="rect"
       mass="0.01"
       update_rate="30"
@@ -51,5 +51,5 @@
       stddev="0.02"
       scale="1.0">
-      <origin xyz="0 0 2" rpy="0 0 0"/>
+      <origin xyz="1 0 2" rpy="0 0 0"/>
       <inertia ixx="0.00001" ixy="0.0" ixz="0.0" iyy="0.00001" iyz="0.0" izz="0.000001"/>
     </xacro:regular_camera_plugin_macro>

Commit message: Finished modding apriltag_ros_config

File: sc_gazebo_plugins/urdf/camera.xacro (robot description, xacro)
@@ -21,5 +21,5 @@
       <xacro:no_collision/>
     </link>
-    <joint name="${namespace}/camer_joint" type="revolute">
+    <joint name="${namespace}/camera_joint" type="revolute">
       <xacro:insert_block name="origin"/>
       <parent link="${parent_link}"/>
@@ -41,9 +41,9 @@
           <cylinder length="0.000001" radius="0.000001"/>
         </geometry>
-        <origin xyz="0 0 0" rpy="0 ${0.5*pi} 0"/>
+        <origin xyz="0 0 0" rpy="0 0 0"/>
       </collision>
     </link>
     <joint name="${namespace}/camera_optical_joint" type="revolute">
-      <origin xyz="0 0 0" rpy="${-pi/2} 0 ${-pi/2}"/>
+      <origin xyz="0 0 0" rpy="0 0 0"/>
       <parent link="${namespace}/camera_link"/>
       <child link="${namespace}/camera_link_optical"/>
