Commit message: Modified inertias for prime, added torque input node, included torque profile script in sc_utils

File: sc_gazebo_plugins/urdf/pose_3d.xacro (robot description, xacro)
@@ -5,6 +5,6 @@
     <link name="${namespace}/pose_sensor_link_${suffix}">
       <inertial>
-        <inertia ixx="0.00001" ixy="0.0" ixz="0.0" iyy="0.00001" iyz="0.0" izz="0.00001"/>
-        <mass value="0.001"/>
+        <inertia ixx="0.000001" ixy="0.0" ixz="0.0" iyy="0.000001" iyz="0.0" izz="0.000001"/>
+        <mass value="0.00001"/>
         <origin xyz="0 0 0" rpy="0 0 0"/>
       </inertial>

File: sc_gazebo_plugins/urdf/reaction_wheel.xacro (robot description, xacro)
@@ -4,8 +4,8 @@
     <link name="${namespace}/wheel_${wheel_id}_link">
       <inertial>
-        <mass value="1"/>
-        <inertia ixx="1" ixy="0.0" ixz="0.0"
-                 iyy="1" iyz="0.0"
-                 izz="1"/>
+        <mass value="0.00001"/>
+        <inertia ixx="0.00001" ixy="0.0" ixz="0.0"
+                 iyy="0.00001" iyz="0.0"
+                 izz="0.00001"/>
       </inertial>
       <visual>

File: urdf/robots/prime_description/urdf/prime_air_bearing.xacro (robot description, xacro)
@@ -3,5 +3,5 @@
   <xacro:macro name="add_bearing" params="namespace bearing_id *origin">
     <link name="${namespace}/bearing_${bearing_id}">
-      <xacro:box_inertial mass="0.0001">
+      <xacro:box_inertial mass="0.000001">
         <xacro:insert_block name="origin"/>
       </xacro:box_inertial>
@@ -41,7 +41,7 @@
       <mass value="${mass}"/>
       <xacro:insert_block name="origin"/>
-      <inertia ixx="0.00001" ixy="0.0" ixz="0.0"
-               iyy="0.00001" iyz="0.0"
-               izz="0.00001"/>
+      <inertia ixx="0.000001" ixy="0.0" ixz="0.0"
+               iyy="0.000001" iyz="0.0"
+               izz="0.000001"/>
     </inertial>
   </xacro:macro>

File: urdf/robots/prime_description/urdf/prime_base.xacro (robot description, xacro)
@@ -47,5 +47,5 @@
         <inertia
           ixx="0.0416833" ixy="0.0" ixz="0.0"
-          iyy="0.0000333" iyz="0.0"
+          iyy="0.0400333" iyz="0.0"
           izz="0.0416833"/>
       </inertial>
