Commit message: Full coordinate two prime torque

File: sc_gazebo_plugins/urdf/basic_lidar.xacro (robot description, xacro)
@@ -25,5 +25,5 @@
     </link>
     <joint name="${namespace}/lidar_sensor_joint" type="fixed">
-      <origin xyz="0 0 1" rpy="0 0 0"/>
+      <origin xyz="0 0 0" rpy="0 0 0"/>
       <parent link="${parent_link}"/>
       <child link="${namespace}/lidar_sensor_link"/>
@@ -31,8 +31,8 @@
     <gazebo reference="${namespace}/lidar_sensor_link">
       <sensor type="gpu_ray" name="${namespace}/lidar_sensor">
-        <always_on>true</always_on>
+        <always_on>false</always_on>
         <update_rate>10</update_rate>
         <pose>0 0 0 0 0 0</pose>
-        <visualize>false</visualize>
+        <visualize>true</visualize>
         <plugin name="pulse_lidar_sensing" filename="libgazebo_ros_velodyne_gpu_laser.so">
           <topicName>lidar_points</topicName>
@@ -46,19 +46,19 @@
           <scan>
             <horizontal>
-              <samples>200</samples>
+              <samples>100</samples>
               <resolution>1</resolution>
-              <min_angle>${-pi/12}</min_angle>
-              <max_angle>${pi/12}</max_angle>
+              <min_angle>${-0.5/12}</min_angle>
+              <max_angle>${0.5/12}</max_angle>
             </horizontal>
             <vertical>
-              <samples>200</samples>
+              <samples>100</samples>
               <resolution>0.1</resolution>
-              <min_angle>${-pi/12}</min_angle>
-              <max_angle>${pi/12}</max_angle>
+              <min_angle>${-0.5/12}</min_angle>
+              <max_angle>${0.5/12}</max_angle>
             </vertical>
           </scan>
           <range>
             <min>0.08</min>
-            <max>20.0</max>
+            <max>2.0</max>
             <resolution>0.01</resolution>
           </range>

File: urdf/robots/prime_description/urdf/prime_base.xacro (robot description, xacro)
@@ -126,4 +126,10 @@
       <origin xyz="0 0 0" rpy="0 0 0"/>
     </xacro:reaction_wheel_macro>
+    <xacro:include filename="$(find sc_gazebo_plugins)/urdf/basic_lidar.xacro"/>
+    <xacro:lidar_macro
+      namespace="${namespace}"
+      parent_link="${namespace}/base_link"
+      inertial_reference_frame="world">
+    </xacro:lidar_macro>
   </xacro:macro>
 </robot>
