Commit message: working on it

File: urdf/robots/cubesat_a_description/urdf/cubesat_base.xacro (robot description, xacro)
@@ -18,5 +18,5 @@
         <origin xyz="0 0 0" rpy="1.570796326794 0 0"/>
         <geometry>
-          <box size="0.1 0.1 0.1"/>
+          <mesh filename="file://$(find cubesat_a_description)/meshes/large_cubesat_female.dae"/>
         </geometry>
       </visual>
@@ -24,5 +24,5 @@
         <origin xyz="0 0 0" rpy="1.570796326794 0 0"/>
         <geometry>
-          <box size="0.1 0.1 0.1"/>
+          <mesh filename="file://$(find cubesat_a_description)/meshes/large_cubesat_female.dae"/>
         </geometry>
       </collision>

File: urdf/robots/cubesat_b_description/urdf/cubesat_base.xacro (robot description, xacro)
@@ -18,5 +18,5 @@
         <origin xyz="0 0 0" rpy="1.570796326794 0 0"/>
         <geometry>
-          <box size="0.1 0.1 0.1"/>
+          <mesh filename="file://$(find cubesat_b_description)/meshes/large_cubesat_male.dae"/>
         </geometry>
       </visual>
@@ -24,5 +24,5 @@
         <origin xyz="0 0 0" rpy="1.570796326794 0 0"/>
         <geometry>
-          <box size="0.1 0.1 0.1"/>
+          <mesh filename="file://$(find cubesat_b_description)/meshes/large_cubesat_male.dae"/>
         </geometry>
       </collision>
