Commit message: Pipeline added for new apriltag additions

File: urdf/robots/cubesat_description/urdf/cubesat_base.xacro (robot description, xacro)
@@ -35,4 +35,32 @@
       <child link="$(arg namespace)/cubesat_link"/>
     </joint>
+    <!-- Create link and joint for apriltag -->
+    <link name="$(arg namespace)/apriltag_link">
+      <inertial>
+        <origin xyz="0 0 0" rpy="0 0 0"/>
+        <mass value="0.0001"/>
+        <inertia
+          ixx="0.0001" ixy="0.0" ixz="0.0"
+          iyy="0.0001" iyz="0.0"
+          izz="0.0001"/>
+      </inertial>
+      <visual>
+        <origin xyz="0.05 0 0" rpy="0 1.57 0"/>
+        <geometry>
+          <mesh filename="package://sc_models/models/apriltags/tag36_11_00000/meshes/tag36_11_00000.dae" scale="0.1 0.1 0.1"/>
+        </geometry>
+      </visual>
+      <collision>
+        <origin xyz="0.05 0 0" rpy="0 1.57 0"/>
+        <geometry>
+          <mesh filename="package://sc_models/models/apriltags/tag36_11_00000/meshes/tag36_11_00000.dae" scale="1 1 1"/>
+        </geometry>
+      </collision>
+    </link>
+    <joint name="$(arg namespace)/apriltag_joint" type="continuous">
+      <origin xyz="0 0 0" rpy="0 0 0"/>
+      <parent link="$(arg namespace)/cubesat_link"/>
+      <child link="$(arg namespace)/apriltag_link"/>
+    </joint>
     <gazebo>
       <plugin name="gazebo_ros_control" filename="libgazebo_ros_control.so">

Commit message: Added granite table model, needs to increase in size

File: urdf/robots/cubesat_description/urdf/cubesat_base.xacro (robot description, xacro)
@@ -35,32 +35,4 @@
       <child link="$(arg namespace)/cubesat_link"/>
     </joint>
-    <!-- Create link and joint for apriltag -->
-    <link name="$(arg namespace)/apriltag_link">
-      <inertial>
-        <origin xyz="0 0 0" rpy="0 0 0"/>
-        <mass value="0.0001"/>
-        <inertia
-          ixx="0.0001" ixy="0.0" ixz="0.0"
-          iyy="0.0001" iyz="0.0"
-          izz="0.0001"/>
-      </inertial>
-      <visual>
-        <origin xyz="0.05 0 0" rpy="0 1.57 0"/>
-        <geometry>
-          <mesh filename="package://sc_models/models/apriltags/tag36_11_00000/meshes/tag36_11_00000.dae" scale="0.1 0.1 0.1"/>
-        </geometry>
-      </visual>
-      <collision>
-        <origin xyz="0.05 0 0" rpy="0 1.57 0"/>
-        <geometry>
-          <mesh filename="package://sc_models/models/apriltags/tag36_11_00000/meshes/tag36_11_00000.dae" scale="1 1 1"/>
-        </geometry>
-      </collision>
-    </link>
-    <joint name="$(arg namespace)/apriltag_joint" type="continuous">
-      <origin xyz="0 0 0" rpy="0 0 0"/>
-      <parent link="$(arg namespace)/cubesat_link"/>
-      <child link="$(arg namespace)/apriltag_link"/>
-    </joint>
     <gazebo>
       <plugin name="gazebo_ros_control" filename="libgazebo_ros_control.so">

Commit message: Think I solved it

File: urdf/robots/cubesat_description/urdf/cubesat_base.xacro (robot description, xacro)
@@ -5,18 +5,20 @@
     <!-- "Dummy base link to eliminate root link inertia warning -->
     <link name="$(arg namespace)/base_link"/>
+    <xacro:property name="side" value="5"/>
+    <xacro:property name="mass" value="10"/>
     <!-- Start of main robot body -->
     <link name="$(arg namespace)/cubesat_link">
       <inertial>
         <origin xyz="0 0 0" rpy="0 0 0"/>
-        <mass value="10.0"/>
+        <mass value="${mass}"/>
         <inertia
-          ixx="10.0" ixy="0.0" ixz="0.0"
-          iyy="10.0" iyz="0.0"
-          izz="10.0"/>
+          ixx="${mass / 12.0 * (side*side + side*side)}" ixy="0.0" ixz="0.0"
+          iyy="${mass / 12.0 * (side*side + side*side)}" iyz="0.0"
+          izz="${mass / 12.0 * (side*side + side*side)}"/>
       </inertial>
       <visual>
         <origin xyz="0 0 0" rpy="1.570796326794 0 0"/>
         <geometry>
-          <box size="0.1 0.1 0.1"/>
+          <box size="${side} ${side} ${side}"/>
         </geometry>
       </visual>
@@ -24,5 +26,5 @@
         <origin xyz="0 0 0" rpy="1.570796326794 0 0"/>
         <geometry>
-          <box size="0.1 0.1 0.1"/>
+          <box size="${side} ${side} ${side}"/>
         </geometry>
       </collision>

File: urdf/robots/prime_description/urdf/prime_base.xacro (robot description, xacro)
@@ -2,4 +2,11 @@
 <robot name="prime" xmlns:xacro="https://www.ros.org/wiki/xacro">
   <xacro:arg name="namespace" default="prime"/>
+  <xacro:property name="PI" value="3.1415926535897931"/>
+  <!--xacro:property name="m1" value="13.0"/-->
+  <xacro:property name="m1" value="13"/>
+  <xacro:property name="m2" value="0.5"/>
+  <xacro:property name="l1" value="0.27"/>
+  <xacro:property name="l2" value="1.0"/>
+  <xacro:property name="l3" value="0.02"/>
   <xacro:macro name="prime_base" params="namespace">
     <!-- "Dummy base link to eliminate root link inertia warning -->
@@ -18,14 +25,19 @@
       <inertial>
         <origin xyz="0 0 0" rpy="0 0 0"/>
-        <mass value="13.0"/>
+        <mass value="${m1}"/>
+        <!--inertia
+          ixx="${(1/6) * m1 * l1 * l1}" ixy="0.0" ixz="0.0"
+          iyy="${(1/6) * m1 * l1 * l1}" iyz="0.0"
+          izz="${(1/6) * m1 * l1 * l1}"/-->
         <inertia
-          ixx="0.15795" ixy="0.0" ixz="0.0"
-          iyy="0.15795" iyz="0.0"
-          izz="0.15795"/>
+          ixx="${m1 / 12 * (l1 * l1 + l1 * l1)}" ixy="0.0" ixz="0.0"
+          iyy="${m1 / 12 * (l1 * l1 + l1 * l1)}" iyz="0.0"
+          izz="${m1 / 12 * (l1 * l1 + l1 * l1)}"/>
       </inertial>
       <visual>
         <origin xyz="0 0 0" rpy="0 0 0"/>
         <geometry>
-          <mesh filename="file://$(find prime_description)/meshes/prime_fss.dae"/>
+          <!--mesh filename="file://$(find prime_description)/meshes/prime_fss.dae"/-->
+          <box size="${l1} ${l1} ${l1}"/>
         </geometry>
       </visual>
@@ -33,5 +45,6 @@
         <origin xyz="0 0 0" rpy="0 0 0"/>
         <geometry>
-          <mesh filename="file://$(find prime_description)/meshes/prime_fss.dae"/>
+          <!--mesh filename="file://$(find prime_description)/meshes/prime_fss.dae"/-->
+          <box size="0.027 0.027 0.027"/>
         </geometry>
       </collision>
@@ -41,5 +54,4 @@
       <origin xyz="0 0 0" rpy="0 0 0"/>
       <parent link="$(arg namespace)/base_link"/>
-      <!--parent link="world"/-->
       <child link="$(arg namespace)/prime_link"/>
     </joint>
@@ -53,20 +65,20 @@
     <link name="$(arg namespace)/mass_bar">
       <inertial>
-        <origin xyz="0 0.5 0.0" rpy="1.57 0 0"/>
-        <mass value="0.5"/>
+        <origin xyz="0 0.5 0.0" rpy="0 0 0"/>
+        <mass value="${m2}"/>
         <inertia
-          ixx="0.0416833" ixy="0.0" ixz="0.0"
-          iyy="0.0400333" iyz="0.0"
-          izz="0.0416833"/>
+          ixx="${(1/12) * m2 * (l2*l2 + l3*l3)}" ixy="0.0" ixz="0.0"
+          iyy="${(1/6) * m2 * l3 * l3}" iyz="0.0"
+          izz="${(1/12) * m2 * (l2*l2 + l3*l3)}"/>
       </inertial>
       <visual>
-        <origin xyz="0 0.5 0" rpy="-1.57 0 0"/>
+        <origin xyz="0 0.5 0.0" rpy="0 0 0"/>
         <geometry>
-          <mesh filename="file://$(find sc_models)/models/grab_solar_panel/meshes/grasp_panel.dae" scale="1 1 0.715"/>
-          <!--box size="0.02 0.02 1.0"/-->
+          <!--mesh filename="file://$(find sc_models)/models/grab_solar_panel/meshes/grasp_panel.dae" scale="1 1 0.715"/-->
+          <box size="0.02 1.0 0.02"/>
         </geometry>
       </visual>
       <collision>
-        <origin xyz="0 0.5 0" rpy="1.57 0 0"/>
+        <origin xyz="0 0.5 0" rpy="0 0 0"/>
         <geometry>
           <box size="0.02 0.02 1.0"/>
@@ -75,10 +87,9 @@
     </link>
     <joint name="$(arg namespace)/torsion_spring_joint" type="revolute">
-      <origin xyz="0 0.135 0.025" rpy="0 0 0"/>
-      <!--origin xyz="0 0.0 0.025" rpy="0 0 0"/-->
+      <origin xyz="0.0 0.135 0.0" rpy="0 0 0"/>
       <parent link="$(arg namespace)/prime_link"/>
       <child link="$(arg namespace)/mass_bar"/>
       <axis xyz="0 0 1"/>
-      <limit effort="100000" lower="-1.57" upper="1.57" velocity="200" />
+      <limit effort="100000" lower="-1.57" upper="1.57" velocity="2000" />
     </joint>
     <gazebo>
@@ -86,5 +97,5 @@
         <torsion_joint>${namespace}/torsion_spring_joint</torsion_joint>
         <kx>0.11</kx>
-        <set_point>0.00000</set_point>
+        <set_point>0.0</set_point>
       </plugin>
     </gazebo>
