Commit message: needs more testing, but looking hopeful for torsion spring plugin

File: urdf/robots/prime_description/urdf/prime_base.xacro (robot description, xacro)
@@ -34,4 +34,41 @@
       <child link="$(arg namespace)/prime_link"/>
     </joint>
+    <!-- Add experimental spring and bar -->
+    <link name="$(arg namespace)/mass_bar">
+      <inertial>
+        <origin xyz="0 0 2" rpy="0 0 0"/>
+        <mass value="1.0"/>
+        <inertia
+          ixx="2.0" ixy="0.0" ixz="0.0"
+          iyy="2.0" iyz="0.0"
+          izz="1.0"/>
+      </inertial>
+      <visual>
+        <origin xyz="0 0 2" rpy="0 0 0"/>
+        <geometry>
+          <box size="0.1 0.1 1.0"/>
+        </geometry>
+      </visual>
+      <collision>
+        <origin xyz="0 0 2" rpy="0 0 0"/>
+        <geometry>
+          <box size="0.1 0.1 1.0"/>
+        </geometry>
+      </collision>
+    </link>
+    <joint name="$(arg namespace)/torsion_spring_joint" type="revolute">
+      <origin xyz="0 0 1.0" rpy="0 0 0"/>
+      <parent link="$(arg namespace)/prime_link"/>
+      <child link="$(arg namespace)/mass_bar"/>
+      <axis xyz="0 0 1"/>
+      <limit effort="0" lower="-1.57" upper="1.57" velocity="0.0"/>
+    </joint>
+    <gazebo>
+      <plugin name="${namespace}_torsion_spring_joint" filename="libsc_torsional_spring_joint_plugin.so">
+        <torsion_joint>${namespace}/torsion_spring_joint</torsion_joint>
+        <kx>0.0</kx>
+        <set_point>0.0</set_point>
+      </plugin>
+    </gazebo>
     <!-- Add air bearings -->
     <xacro:include filename="$(find prime_description)/urdf/prime_air_bearing.xacro"/>

Commit message: Modifying torsional spring plugin to advertise spring angle

File: urdf/robots/prime_description/urdf/prime_base.xacro (robot description, xacro)
@@ -34,38 +34,44 @@
       <child link="$(arg namespace)/prime_link"/>
     </joint>
+    <!-- Connect base to world, fixed -->
+    <joint name="$(arg namespace)/world_fixed" type="fixed">
+      <origin xyz="0 0 0" rpy="0 0 0"/>
+      <parent link="world"/>
+      <child link="$(arg namespace)/base_link"/>
+    </joint>
     <!-- Add experimental spring and bar -->
     <link name="$(arg namespace)/mass_bar">
       <inertial>
-        <origin xyz="0 0 2" rpy="0 0 0"/>
-        <mass value="1.0"/>
+        <origin xyz="0 0.45 0" rpy="1.57 0 0"/>
+        <mass value="2.0"/>
         <inertia
-          ixx="2.0" ixy="0.0" ixz="0.0"
-          iyy="2.0" iyz="0.0"
-          izz="1.0"/>
+          ixx="0.5" ixy="0.0" ixz="0.0"
+          iyy="0.5" iyz="0.0"
+          izz="0.25"/>
       </inertial>
       <visual>
-        <origin xyz="0 0 2" rpy="0 0 0"/>
+        <origin xyz="0 0.45 0" rpy="1.57 0 0"/>
         <geometry>
-          <box size="0.1 0.1 1.0"/>
+          <box size="0.05 0.05 0.5"/>
         </geometry>
       </visual>
       <collision>
-        <origin xyz="0 0 2" rpy="0 0 0"/>
+        <origin xyz="0 0.45 0" rpy="1.57 0 0"/>
         <geometry>
-          <box size="0.1 0.1 1.0"/>
+          <box size="0.05 0.05 0.5"/>
         </geometry>
       </collision>
     </link>
     <joint name="$(arg namespace)/torsion_spring_joint" type="revolute">
-      <origin xyz="0 0 1.0" rpy="0 0 0"/>
+      <origin xyz="0 0 0.0" rpy="0 0 0"/>
       <parent link="$(arg namespace)/prime_link"/>
       <child link="$(arg namespace)/mass_bar"/>
       <axis xyz="0 0 1"/>
-      <limit effort="0" lower="-1.57" upper="1.57" velocity="0.0"/>
+      <limit effort="100000" lower="-1.57" upper="1.57" velocity="0.0"/>
     </joint>
     <gazebo>
       <plugin name="${namespace}_torsion_spring_joint" filename="libsc_torsional_spring_joint_plugin.so">
         <torsion_joint>${namespace}/torsion_spring_joint</torsion_joint>
-        <kx>0.0</kx>
+        <kx>0.5</kx>
         <set_point>0.0</set_point>
       </plugin>

Commit message: Completed setting up prime experiment

File: urdf/robots/prime_description/urdf/prime_base.xacro (robot description, xacro)
@@ -34,15 +34,15 @@
       <child link="$(arg namespace)/prime_link"/>
     </joint>
-    <!-- Connect base to world, fixed -->
+    <!-- Connect base to world, fixed >
     <joint name="$(arg namespace)/world_fixed" type="fixed">
       <origin xyz="0 0 0" rpy="0 0 0"/>
       <parent link="world"/>
       <child link="$(arg namespace)/base_link"/>
-    </joint>
+    </joint-->
     <!-- Add experimental spring and bar -->
     <link name="$(arg namespace)/mass_bar">
       <inertial>
         <origin xyz="0 0.45 0" rpy="1.57 0 0"/>
-        <mass value="2.0"/>
+        <mass value="2"/>
         <inertia
           ixx="0.5" ixy="0.0" ixz="0.0"
@@ -64,15 +64,15 @@
     </link>
     <joint name="$(arg namespace)/torsion_spring_joint" type="revolute">
-      <origin xyz="0 0 0.0" rpy="0 0 0"/>
+      <origin xyz="0 0 0" rpy="0 0 0"/>
       <parent link="$(arg namespace)/prime_link"/>
       <child link="$(arg namespace)/mass_bar"/>
       <axis xyz="0 0 1"/>
-      <limit effort="100000" lower="-1.57" upper="1.57" velocity="0.0"/>
+      <limit effort="100000" lower="-1.57" upper="1.57" velocity="200" />
     </joint>
     <gazebo>
       <plugin name="${namespace}_torsion_spring_joint" filename="libsc_torsional_spring_joint_plugin.so">
         <torsion_joint>${namespace}/torsion_spring_joint</torsion_joint>
-        <kx>0.5</kx>
-        <set_point>0.0</set_point>
+        <kx>0.1</kx>
+        <set_point>0.2</set_point>
       </plugin>
     </gazebo>

Commit message: Adjusted prime and mass parameters for experiment

File: urdf/robots/prime_description/urdf/prime_base.xacro (robot description, xacro)
@@ -9,5 +9,5 @@
       <inertial>
         <origin xyz="0 0 0" rpy="0 0 0"/>
-        <mass value="50.0"/>
+        <mass value="13.0"/>
         <inertia
           ixx="30.0" ixy="0.0" ixz="0.0"
@@ -43,6 +43,6 @@
     <link name="$(arg namespace)/mass_bar">
       <inertial>
-        <origin xyz="0 0.45 0" rpy="1.57 0 0"/>
-        <mass value="2"/>
+        <origin xyz="0 0.5 0.0" rpy="1.57 0 0"/>
+        <mass value="0.5"/>
         <inertia
           ixx="0.5" ixy="0.0" ixz="0.0"
@@ -51,18 +51,18 @@
       </inertial>
       <visual>
-        <origin xyz="0 0.45 0" rpy="1.57 0 0"/>
+        <origin xyz="0 0.5 0" rpy="1.57 0 0"/>
         <geometry>
-          <box size="0.05 0.05 0.5"/>
+          <box size="0.02 0.02 1.0"/>
         </geometry>
       </visual>
       <collision>
-        <origin xyz="0 0.45 0" rpy="1.57 0 0"/>
+        <origin xyz="0 0.5 0" rpy="1.57 0 0"/>
         <geometry>
-          <box size="0.05 0.05 0.5"/>
+          <box size="0.02 0.02 1.0"/>
         </geometry>
       </collision>
     </link>
     <joint name="$(arg namespace)/torsion_spring_joint" type="revolute">
-      <origin xyz="0 0 0" rpy="0 0 0"/>
+      <origin xyz="0 0.135 0.025" rpy="0 0 0"/>
       <parent link="$(arg namespace)/prime_link"/>
       <child link="$(arg namespace)/mass_bar"/>
@@ -73,6 +73,6 @@
       <plugin name="${namespace}_torsion_spring_joint" filename="libsc_torsional_spring_joint_plugin.so">
         <torsion_joint>${namespace}/torsion_spring_joint</torsion_joint>
-        <kx>0.1</kx>
-        <set_point>0.2</set_point>
+        <kx>0.11</kx>
+        <set_point>0.05</set_point>
       </plugin>
     </gazebo>

Commit message: Added solar panel to prime experiment

File: urdf/robots/prime_description/urdf/prime_base.xacro (robot description, xacro)
@@ -51,7 +51,8 @@
       </inertial>
       <visual>
-        <origin xyz="0 0.5 0" rpy="1.57 0 0"/>
+        <origin xyz="0 0.5 0" rpy="-1.57 0 0"/>
         <geometry>
-          <box size="0.02 0.02 1.0"/>
+          <mesh filename="file://$(find sc_models)/models/grab_solar_panel/meshes/grasp_panel.dae" scale="1 1 0.715"/>
+          <!--box size="0.02 0.02 1.0"/-->
         </geometry>
       </visual>

Commit message: Added two primes to environment, adjusted sun position

File: urdf/robots/prime_description/urdf/prime_base.xacro (robot description, xacro)
@@ -71,4 +71,32 @@
       <limit effort="100000" lower="-1.57" upper="1.57" velocity="200" />
     </joint>
+    <!--link name="$(arg namespace)/direction_beam">
+      <inertial>
+        <origin xyz="0 0 0" rpy="0 0 0"/>
+        <mass value="0.001"/>
+        <inertia
+          ixx="0.001" ixy="0.0" ixz="0.0"
+          iyy="0.001" iyz="0.0"
+          izz="0.001"/>
+      </inertial>
+      <visual>
+        <origin xyz="0 0 0" rpy="0 0 0"/>
+        <geometry>
+          <cylinder radius="0.01" length="1.0"/>
+        </geometry>
+      </visual>
+      <collision>
+        <origin xyz="0 0 0" rpy="0 0 0"/>
+        <geometry>
+          <cylinder radius="0.000001" length="0.00001"/>
+        </geometry>
+      </collision>
+    </link>
+    <joint name="$(arg namespace)/direction_beam_joint" type="revolute">
+      <origin xyz="0.135 0 0.025" rpy="0 1.57 0"/>
+      <parent link="$(arg namespace)/prime_link"/>
+      <child link="$(arg namespace)/direction_beam"/>
+      <limit effort="100000" lower="0" upper="0" velocity="200" />
+    </joint-->
     <gazebo>
       <plugin name="${namespace}_torsion_spring_joint" filename="libsc_torsional_spring_joint_plugin.so">

Commit message: Modified mass and I values for Clouse experiment

File: urdf/robots/prime_description/urdf/prime_base.xacro (robot description, xacro)
@@ -4,4 +4,5 @@
   <xacro:macro name="prime_base" params="namespace">
     <!-- "Dummy base link to eliminate root link inertia warning -->
+    <!--https://dynref.engr.illinois.edu/rem.html-->
     <link name="$(arg namespace)/base_link"/>
     <!-- Start of main robot body -->
@@ -9,5 +10,6 @@
       <inertial>
         <origin xyz="0 0 0" rpy="0 0 0"/>
-        <mass value="13.0"/>
+        <mass value="10.0"/>
+          <!-- I = 0.1215 -->
         <inertia
           ixx="0.15795" ixy="0.0" ixz="0.0"
@@ -44,5 +46,6 @@
       <inertial>
         <origin xyz="0 0.5 0.0" rpy="1.57 0 0"/>
-        <mass value="0.5"/>
+        <mass value="2"/>
+          <!--I=0.0266708 -->
         <inertia
           ixx="0.0416833" ixy="0.0" ixz="0.0"
@@ -53,6 +56,5 @@
         <origin xyz="0 0.5 0" rpy="-1.57 0 0"/>
         <geometry>
-          <mesh filename="file://$(find sc_models)/models/grab_solar_panel/meshes/grasp_panel.dae" scale="1 1 0.715"/>
-          <!--box size="0.02 0.02 1.0"/-->
+          <box size="0.005 0.005 0.4"/>
         </geometry>
       </visual>
@@ -60,5 +62,5 @@
         <origin xyz="0 0.5 0" rpy="1.57 0 0"/>
         <geometry>
-          <box size="0.02 0.02 1.0"/>
+          <box size="0.005 0.005 0.4"/>
         </geometry>
       </collision>
@@ -74,5 +76,5 @@
       <plugin name="${namespace}_torsion_spring_joint" filename="libsc_torsional_spring_joint_plugin.so">
         <torsion_joint>${namespace}/torsion_spring_joint</torsion_joint>
-        <kx>0.11</kx>
+        <kx>0.5</kx>
         <set_point>0.0</set_point>
       </plugin>

Commit message: Modified data read

File: urdf/robots/prime_description/urdf/prime_base.xacro (robot description, xacro)
@@ -13,7 +13,7 @@
           <!-- I = 0.1215 -->
         <inertia
-          ixx="0.15795" ixy="0.0" ixz="0.0"
-          iyy="0.15795" iyz="0.0"
-          izz="0.15795"/>
+          ixx="0.1215" ixy="0.0" ixz="0.0"
+          iyy="0.1215" iyz="0.0"
+          izz="0.1215"/>
       </inertial>
       <visual>
@@ -45,22 +45,23 @@
     <link name="$(arg namespace)/mass_bar">
       <inertial>
-        <origin xyz="0 0.5 0.0" rpy="1.57 0 0"/>
+        <origin xyz="0 0.2 0.0" rpy="0 0 0"/>
         <mass value="2"/>
           <!--I=0.0266708 -->
         <inertia
-          ixx="0.0416833" ixy="0.0" ixz="0.0"
-          iyy="0.0400333" iyz="0.0"
-          izz="0.0416833"/>
+          ixx="0.0266708" ixy="0.0" ixz="0.0"
+          iyy="0.0266708" iyz="0.0"
+          izz="0.0266708"/>
       </inertial>
+      <!-- iyy="0.000008333" iyz="0.0"-->
       <visual>
-        <origin xyz="0 0.5 0" rpy="-1.57 0 0"/>
+        <origin xyz="0 0.2 0" rpy="0 0 0"/>
         <geometry>
-          <box size="0.005 0.005 0.4"/>
+          <box size="0.005 0.4 0.005"/>
         </geometry>
       </visual>
       <collision>
-        <origin xyz="0 0.5 0" rpy="1.57 0 0"/>
+        <origin xyz="0 0.2 0" rpy="0 0 0"/>
         <geometry>
-          <box size="0.005 0.005 0.4"/>
+          <box size="0.005 0.4 0.005"/>
         </geometry>
       </collision>

Commit message: update the mess

File: urdf/robots/prime_description/urdf/prime_base.xacro (robot description, xacro)
@@ -5,4 +5,13 @@
     <!-- "Dummy base link to eliminate root link inertia warning -->
     <link name="$(arg namespace)/base_link"/>
+    <!--link name="world"/-->
+    <!--joint name="$(arg namespace)/world_joint" type="continuous">
+      <origin xyz="0 0 0" rpy="0 0 0"/>
+      <parent link="world"/>
+      <child link="$(arg namespace)/base_link"/>
+      <axis>
+        <xyz>0 0 1</xyz>
+      </axis>
+    </joint-->
     <!-- Start of main robot body -->
     <link name="$(arg namespace)/prime_link">
@@ -32,4 +41,5 @@
       <origin xyz="0 0 0" rpy="0 0 0"/>
       <parent link="$(arg namespace)/base_link"/>
+      <!--parent link="world"/-->
       <child link="$(arg namespace)/prime_link"/>
     </joint>
@@ -66,4 +76,5 @@
     <joint name="$(arg namespace)/torsion_spring_joint" type="revolute">
       <origin xyz="0 0.135 0.025" rpy="0 0 0"/>
+      <!--origin xyz="0 0.0 0.025" rpy="0 0 0"/-->
       <parent link="$(arg namespace)/prime_link"/>
       <child link="$(arg namespace)/mass_bar"/>
@@ -78,4 +89,17 @@
       </plugin>
     </gazebo>
+    <!--gazebo>
+    <joint name="prime_riser" type="prismatic">
+      <parent>world</parent>
+      <child>prime/base_link</child>
+      <axis>
+        <limit>
+          <lower>0</lower>
+          <upper>2</upper>
+        </limit>
+        <xyz>0 0 1</xyz>
+      </axis>
+    </joint>
+  </gazebo-->
     <gazebo>
       <plugin name="${namespace}_initial_velocity" filename="libsc_set_initial_velocity_plugin.so">
@@ -83,5 +107,5 @@
     </gazebo>
     <!-- Add air bearings -->
-    <xacro:include filename="$(find prime_description)/urdf/prime_air_bearing.xacro"/>
+    <!--xacro:include filename="$(find prime_description)/urdf/prime_air_bearing.xacro"/>
     <xacro:add_bearing namespace="${namespace}" bearing_id="0">
       <origin xyz="0 ${0.27/2-0.05/2} ${-0.25-0.005}" rpy="0 0 0"/>
@@ -92,5 +116,5 @@
     <xacro:add_bearing namespace="${namespace}" bearing_id="2">
       <origin xyz="${-0.27/2+0.05/2} -${0.27/2-0.05/2} ${-0.25-0.005}" rpy="0 0 0"/>
-    </xacro:add_bearing>
+    </xacro:add_bearing-->
     <gazebo>
       <plugin name="gazebo_ros_control" filename="libgazebo_ros_control.so">
@@ -98,8 +122,8 @@
     </gazebo>
     <xacro:arg name="inertial_reference_frame" default="world"/>
-    <xacro:include filename="$(find sc_gazebo_plugins)/urdf/reaction_wheel.xacro"/>
+    <!--xacro:include filename="$(find sc_gazebo_plugins)/urdf/reaction_wheel.xacro"/>
     <xacro:reaction_wheel_macro namespace="$(arg namespace)" wheel_id="0">
       <origin xyz="0 0 0" rpy="0 0 0"/>
-    </xacro:reaction_wheel_macro>
+    </xacro:reaction_wheel_macro-->
   </xacro:macro>
 </robot>

File: urdf/robots/prime_description/urdf/prime_robot.urdf.xacro (robot description, xacro)
@@ -8,15 +8,15 @@
   <xacro:include filename="$(find prime_description)/urdf/prime_base.xacro"/>
   <xacro:prime_base namespace="$(arg namespace)"/>
-  <xacro:include filename="$(find sc_gazebo_plugins)/urdf/imu.xacro"/>
+  <!--xacro:include filename="$(find sc_gazebo_plugins)/urdf/imu.xacro"/>
   <xacro:default_imu_macro
     namespace="$(arg namespace)"
-    parent_link="$(arg namespace)/base_link"
+    parent_link="$(arg namespace)/prime_link"
     inertial_reference_frame="$(arg inertial_reference_frame)">
     <origin xyz="0 0 0" rpy="0 0 0"/>
-  </xacro:default_imu_macro>
+  </xacro:default_imu_macro-->
   <xacro:include filename="$(find sc_gazebo_plugins)/urdf/pose_3d.xacro"/>
   <xacro:default_pose_3d
     namespace="$(arg namespace)"
-    parent_link="$(arg namespace)/base_link">
+    parent_link="$(arg namespace)/prime_link">
   </xacro:default_pose_3d>
   <!--xacro:include filename="$(find prime_description)/urdf/prime_reaction_wheels.xacro"/>

Commit message: Updated of simplified, from set initital conditions

File: urdf/robots/prime_description/urdf/prime_base.xacro (robot description, xacro)
@@ -12,13 +12,4 @@
     <!-- "Dummy base link to eliminate root link inertia warning -->
     <link name="$(arg namespace)/base_link"/>
-    <!--link name="world"/-->
-    <!--joint name="$(arg namespace)/world_joint" type="continuous">
-      <origin xyz="0 0 0" rpy="0 0 0"/>
-      <parent link="world"/>
-      <child link="$(arg namespace)/base_link"/>
-      <axis>
-        <xyz>0 0 1</xyz>
-      </axis>
-    </joint-->
     <!-- Start of main robot body -->
     <link name="$(arg namespace)/prime_link">
@@ -26,8 +17,4 @@
         <origin xyz="0 0 0" rpy="0 0 0"/>
         <mass value="${m1}"/>
-        <!--inertia
-          ixx="${(1/6) * m1 * l1 * l1}" ixy="0.0" ixz="0.0"
-          iyy="${(1/6) * m1 * l1 * l1}" iyz="0.0"
-          izz="${(1/6) * m1 * l1 * l1}"/-->
         <inertia
           ixx="${m1 / 12 * (l1 * l1 + l1 * l1)}" ixy="0.0" ixz="0.0"
@@ -38,6 +25,6 @@
         <origin xyz="0 0 0" rpy="0 0 0"/>
         <geometry>
-          <!--mesh filename="file://$(find prime_description)/meshes/prime_fss.dae"/-->
-          <box size="${l1} ${l1} ${l1}"/>
+          <mesh filename="file://$(find prime_description)/meshes/prime_fss.dae"/>
+          <!--box size="${l1} ${l1} ${l1}"/-->
         </geometry>
       </visual>
@@ -73,8 +60,8 @@
       </inertial>
       <visual>
-        <origin xyz="0 0.5 0.0" rpy="0 0 0"/>
+        <origin xyz="0 0.5 0.0" rpy="${-PI/2} 0 0"/>
         <geometry>
-          <!--mesh filename="file://$(find sc_models)/models/grab_solar_panel/meshes/grasp_panel.dae" scale="1 1 0.715"/-->
-          <box size="0.02 1.0 0.02"/>
+          <mesh filename="file://$(find sc_models)/models/grab_solar_panel/meshes/grasp_panel.dae" scale="1 1 0.715"/>
+          <!--box size="0.02 1.0 0.02"/-->
         </geometry>
       </visual>
@@ -82,5 +69,5 @@
         <origin xyz="0 0.5 0" rpy="0 0 0"/>
         <geometry>
-          <box size="0.02 0.02 1.0"/>
+          <box size="0.002 0.002 0.002"/>
         </geometry>
       </collision>
